File: HDK/HMI.kicad_sch (KiCad schematic)
At the start: 39 parts, among them J401 USB_C, J402 MicroFit_02x10V-H, J403 PH_01x05V-H, J404 PH_01x05V-H, J405 PH_01x05V-H, J406 PH_01x05V-H, J407 PH_01x05V-H, J408 PH_01x05V-H, J409 PH_01x05V-H, J410 PH_01x05V-H, J411 PH_01x05V-H, J412 PH_01x05V-H, J413 PHD_02x04V-H, J414 PHD_02x04V-H, J415 2.54mm2x20V-H, J416 PH_01x05V-H, J417 PHD_02x04V-H, SW401 SW_Push, SW402 SW_Push, SW403 SW_Push, SW404 SW_Push

Commit message: fixed bom
Parts:
- H401, H402, H403, H404: now left out of the parts list
Changed lines of the file:
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@@
+    )
+  )
+  (symbol (lib_id "Mechanical:MountingHole_Pad") (at 41.91 176.53 0) (unit 1)
+    (in_bom no) (on_board yes) (dnp no)
+    (property "Reference" "H403" (at 38.1 168.91 0)
+      (effects (font (size 1.27 1.27)) (justify left))
+    )
+    (property "Value" "M4 Pad" (at 38.1 171.45 0)
+      (effects (font (size 1.27 1.27)) (justify left))
+    )
+    (property "Footprint" "MountingHole:MountingHole_4.3mm_M4_DIN965_Pad_TopBottom" (at 41.91 176.53 0)
+      (effects (font (size 1.27 1.27)) hide)
+    )
+    (property "Datasheet" "~" (at 41.91 176.53 0)
+      (effects (font (size 1.27 1.27)) hide)
+    )
+    (property "LCSC" "-" (at 41.91 176.53 0)
+      (effects (font (size 1.27 1.27)) hide)
+    )
+    (pin "1")
+    (instances
+      (project "bigger-brain"
+        (path "/4f585eb3-0717-4acd-9fc1-ccc573c80f45/a2e49620-6bcb-48ed-bf4e-cee4a2fe5c52"
+          (reference "H403") (unit 1)
+        )
+      )
     )
   )
@@
         (path "/4f585eb3-0717-4acd-9fc1-ccc573c80f45/a2e49620-6bcb-48ed-bf4e-cee4a2fe5c52"
           (reference "#PWR0403") (unit 1)
-        )
-      )
-    )
-  )
-  (symbol (lib_id "Mechanical:MountingHole_Pad") (at 41.91 176.53 0) (unit 1)
-    (in_bom yes) (on_board yes) (dnp no)
-    (property "Reference" "H403" (at 38.1 168.91 0)
-      (effects (font (size 1.27 1.27)) (justify left))
-    )
-    (property "Value" "M4 Pad" (at 38.1 171.45 0)
-      (effects (font (size 1.27 1.27)) (justify left))
-    )
-    (property "Footprint" "MountingHole:MountingHole_4.3mm_M4_DIN965_Pad_TopBottom" (at 41.91 176.53 0)
-      (effects (font (size 1.27 1.27)) hide)
-    )
-    (property "Datasheet" "~" (at 41.91 176.53 0)
-      (effects (font (size 1.27 1.27)) hide)
-    )
-    (property "LCSC" "-" (at 41.91 176.53 0)
-      (effects (font (size 1.27 1.27)) hide)
-    )
-    (pin "1")
-    (instances
-      (project "bigger-brain"
-        (path "/4f585eb3-0717-4acd-9fc1-ccc573c80f45/a2e49620-6bcb-48ed-bf4e-cee4a2fe5c52"
-          (reference "H403") (unit 1)
         )
       )
@@
     )
   )
+  (symbol (lib_id "Mechanical:MountingHole_Pad") (at 50.8 176.53 0) (unit 1)
+    (in_bom no) (on_board yes) (dnp no)
+    (property "Reference" "H404" (at 46.99 168.91 0)
+      (effects (font (size 1.27 1.27)) (justify left))
+    )
+    (property "Value" "M4 Pad" (at 46.99 171.45 0)
+      (effects (font (size 1.27 1.27)) (justify left))
+    )
+    (property "Footprint" "MountingHole:MountingHole_4.3mm_M4_DIN965_Pad_TopBottom" (at 50.8 176.53 0)
+      (effects (font (size 1.27 1.27)) hide)
+    )
+    (property "Datasheet" "~" (at 50.8 176.53 0)
+      (effects (font (size 1.27 1.27)) hide)
+    )
+    (property "LCSC" "-" (at 50.8 176.53 0)
+      (effects (font (size 1.27 1.27)) hide)
+    )
+    (pin "1")
+    (instances
+      (project "bigger-brain"
+        (path "/4f585eb3-0717-4acd-9fc1-ccc573c80f45/a2e49620-6bcb-48ed-bf4e-cee4a2fe5c52"
+          (reference "H404") (unit 1)
+        )
+      )
+    )
+  )
   (symbol (lib_id "power:+3V3") (at 148.59 86.36 270) (unit 1)
     (in_bom yes) (on_board yes) (dnp no) (fields_autoplaced)
@@
     )
   )
-  (symbol (lib_id "Mechanical:MountingHole_Pad") (at 50.8 176.53 0) (unit 1)
-    (in_bom yes) (on_board yes) (dnp no)
-    (property "Reference" "H404" (at 46.99 168.91 0)
-      (effects (font (size 1.27 1.27)) (justify left))
-    )
-    (property "Value" "M4 Pad" (at 46.99 171.45 0)
-      (effects (font (size 1.27 1.27)) (justify left))
-    )
-    (property "Footprint" "MountingHole:MountingHole_4.3mm_M4_DIN965_Pad_TopBottom" (at 50.8 176.53 0)
-      (effects (font (size 1.27 1.27)) hide)
-    )
-    (property "Datasheet" "~" (at 50.8 176.53 0)
-      (effects (font (size 1.27 1.27)) hide)
-    )
-    (property "LCSC" "-" (at 50.8 176.53 0)
-      (effects (font (size 1.27 1.27)) hide)
-    )
-    (pin "1")
-    (instances
-      (project "bigger-brain"
-        (path "/4f585eb3-0717-4acd-9fc1-ccc573c80f45/a2e49620-6bcb-48ed-bf4e-cee4a2fe5c52"
-          (reference "H404") (unit 1)
-        )
-      )
-    )
-  )
   (symbol (lib_id "Device:D_Schottky") (at 87.63 25.4 180) (unit 1)
     (in_bom yes) (on_board yes) (dnp no)
@@
         (path "/4f585eb3-0717-4acd-9fc1-ccc573c80f45/a2e49620-6bcb-48ed-bf4e-cee4a2fe5c52"
           (reference "#PWR0411") (unit 1)
+        )
+      )
+    )
+  )
+  (symbol (lib_id "Mechanical:MountingHole_Pad") (at 33.02 176.53 0) (unit 1)
+    (in_bom no) (on_board yes) (dnp no)
+    (property "Reference" "H402" (at 29.21 168.91 0)
+      (effects (font (size 1.27 1.27)) (justify left))
+    )
+    (property "Value" "M4 Pad" (at 29.21 171.45 0)
+      (effects (font (size 1.27 1.27)) (justify left))
+    )
+    (property "Footprint" "MountingHole:MountingHole_4.3mm_M4_DIN965_Pad_TopBottom" (at 33.02 176.53 0)
+      (effects (font (size 1.27 1.27)) hide)
+    )
+    (property "Datasheet" "~" (at 33.02 176.53 0)
+      (effects (font (size 1.27 1.27)) hide)
+    )
+    (property "LCSC" "-" (at 33.02 176.53 0)
+      (effects (font (size 1.27 1.27)) hide)
+    )
+    (pin "1")
+    (instances
+      (project "bigger-brain"
+        (path "/4f585eb3-0717-4acd-9fc1-ccc573c80f45/a2e49620-6bcb-48ed-bf4e-cee4a2fe5c52"
+          (reference "H402") (unit 1)
         )
       )
@@
   )
   (symbol (lib_id "Mechanical:MountingHole_Pad") (at 24.13 176.53 0) (unit 1)
-    (in_bom yes) (on_board yes) (dnp no)
+    (in_bom no) (on_board yes) (dnp no)
     (property "Reference" "H401" (at 20.32 168.91 0)
       (effects (font (size 1.27 1.27)) (justify left))
@@
         )
       )
-    )
-  )
-  (symbol (lib_id "Mechanical:MountingHole_Pad") (at 33.02 176.53 0) (unit 1)
-    (in_bom yes) (on_board yes) (dnp no)
-    (property "Reference" "H402" (at 29.21 168.91 0)
-      (effects (font (size 1.27 1.27)) (justify left))
-    )
-    (property "Value" "M4 Pad" (at 29.21 171.45 0)
-      (effects (font (size 1.27 1.27)) (justify left))
-    )
-    (property "Footprint" "MountingHole:MountingHole_4.3mm_M4_DIN965_Pad_TopBottom" (at 33.02 176.53 0)
-      (effects (font (size 1.27 1.27)) hide)
-    )
-    (property "Datasheet" "~" (at 33.02 176.53 0)
-      (effects (font (size 1.27 1.27)) hide)
-    )
-    (property "LCSC" "-" (at 33.02 176.53 0)
-      (effects (font (size 1.27 1.27)) hide)
-    )
-    (pin "1")
-    (instances
-      (project "bigger-brain"
-        (path "/4f585eb3-0717-4acd-9fc1-ccc573c80f45/a2e49620-6bcb-48ed-bf4e-cee4a2fe5c52"
-          (reference "H402") (unit 1)
-        )
-      )
