File: HDK/HMI.kicad_sch (KiCad schematic)
At the start: 9 parts, among them J101 USB_C_Receptacle_USB2.0, J402 Conn_02x12_Top_Bottom, U401 74HC245

Commit message: updated WIP
Parts:
- added D401, D402: D_Schottky, symbol Device:D_Schottky
- added J403, J404, J405: Conn_01x03, symbol Connector_Generic:Conn_01x03
- J402: footprint Connector_Molex:Molex_Mini-Fit_Jr_5566-24A_2x12_P4.20mm_Vertical -> NVF-Kicad-Resources:Micro-Fit_2x12V-H
- renumbered C101 to C401, J101 to J401, R101 to R401, R102 to R402
Connections:
- net +5V: now also D401.1 (K), J403.1 (Pin_1), J404.1 (Pin_1), J405.1 (Pin_1)
- net DET1_A: now also U401.8 (A6)
- net DET2_A: now also U401.9 (A7)
- net DET3_A: now also U401.7 (A5)
- net GND: now also J403.3 (Pin_3), J404.3 (Pin_3), J405.3 (Pin_3)
- net VBUS: now also D401.2 (A), D402.2 (A)
- new net 5V_PWM1: J403.2 (Pin_2)
- new net 5V_PWM2: J404.2 (Pin_2)
- new net 5V_PWM3: J405.2 (Pin_2)
- new net VCC: D402.1 (K)

Commit message: added rev1-final
Parts:
- removed J402: Conn_02x12_Top_Bottom, NVF-Kicad-Resources:Micro-Fit_2x12V-H, symbol Connector_Generic:Conn_02x12_Top_Bottom
- removed J403, J404, J405: Conn_01x03, symbol Connector_Generic:Conn_01x03
- removed U401: 74HC245, Package_SO:TSSOP-20_4.4x6.5mm_P0.65mm, symbol 74xx:74HC245
- added C402, C403: 100n, Capacitor_SMD:C_0603_1608Metric, symbol Device:C
- added H401, H402, H403, H404: M4 Pad, MountingHole:MountingHole_4.3mm_M4_DIN965_Pad_TopBottom, symbol Mechanical:MountingHole_Pad
- added J402: MicroFit_02x10V-H, NVF-Kicad:MicroFit_02x10V-H, symbol Connector_Generic:Conn_02x10_Top_Bottom
- added J403, J404, J405, J406, J407, J408, J409, J410, J411, J412, J416: PH_01x05V-H, NVF-Kicad:PH_01x05V-H, symbol Connector_Generic:Conn_01x05
- added J413, J414, J417: PHD_02x04V-H, NVF-Kicad:PHD_02x04V-H, symbol Connector_Generic:Conn_02x04_Odd_Even
- added J415: 2.54mm2x20V-H, NVF-Kicad:2.54mm2x20V-H, symbol Connector_Generic:Conn_02x20_Odd_Even
- added R406, R407, R408: 10k, Resistor_SMD:R_0603_1608Metric, symbol Device:R
- added SW401, SW402, SW403, SW404: SW_Push, NVF-Kicad:PushBtn_TS-1187A-B-A-B, symbol Switch:SW_Push
- added SWD401: ~, NVF-Kicad:2.54mm2x04V-H, symbol NVF-Kicad:SWD_Breakout
- C401: LCSC C57112 -> C14663
- D401, D402: value D_Schottky -> SS14; footprint (none) -> Diode_SMD:D_SMA; LCSC (none) -> C2480
- J401: value USB_C_Receptacle_USB2.0 -> USB_C; footprint NVF-Kicad:USB_C_Receptacle_HRO_TYPE-C-31-M-12 -> NVF-Kicad:USBC_HRO_TYPE-C-31-M-12
- R403, R404, R405: LCSC (none) -> C17909
Connections:
- net +5V: now also J403.1 (Pin_1), J404.1 (Pin_1), J405.1 (Pin_1), J406.1 (Pin_1), J407.1 (Pin_1), J408.1 (Pin_1), J409.1 (Pin_1), J410.1 (Pin_1), J411.1 (Pin_1), J412.1 (Pin_1), J413.1 (Pin_1), J414.1 (Pin_1), J415.31 (Pin_31), J415.32 (Pin_32), J416.1 (Pin_1), J417.1 (Pin_1); no longer C401.1
- net CAN1_H: now also J402.15 (Pin_15), J402.5 (Pin_5)
- net CAN1_L: now also J402.4 (Pin_4)
- net CAN1_L-T: now also J402.14 (Pin_14)
- net CAN2_H: now also J402.12 (Pin_12), J402.2 (Pin_2)
- net CAN2_L: now also J402.1 (Pin_1)
- net CAN2_L-T: now also J402.11 (Pin_11)
- net CAN3_H: now also J402.18 (Pin_18), J402.8 (Pin_8)
- net CAN3_L: now also J402.7 (Pin_7)
- net CAN3_L-T: now also J402.17 (Pin_17)
- net GND: now also C402.2, C403.2, H401.1, H402.1, H403.1, H404.1, J402.13 (Pin_13), J402.16 (Pin_16), J402.19 (Pin_19), J402.20 (Pin_20), J402.6 (Pin_6), J403.5 (Pin_5), J404.5 (Pin_5), J405.5 (Pin_5), J406.5 (Pin_5), J407.5 (Pin_5), J408.5 (Pin_5), J409.5 (Pin_5), J410.5 (Pin_5), J411.5 (Pin_5), J412.5 (Pin_5), J413.7 (Pin_7), J414.7 (Pin_7), J415.33 (Pin_33), J415.34 (Pin_34), J415.37 (Pin_37), J415.38 (Pin_38), J416.5 (Pin_5), J417.7 (Pin_7), R406.2, SW402.2, SW403.2, SW404.2, SWD401.7 (GND), SWD401.8 (GND)
- net PWM1: now also J403.3 (Pin_3)
- net PWM2: now also J403.4 (Pin_4)
- net PWM3: now also J404.4 (Pin_4)
- net PWM4: now also J404.3 (Pin_3)
- net V1: now also J402.9 (Pin_9)
- net V2: now also J402.10 (Pin_10)
- net VCC: now also J415.39 (Pin_39), J415.40 (Pin_40)
- new net +3V3: J403.2 (Pin_2), J404.2 (Pin_2), J405.2 (Pin_2), J406.2 (Pin_2), J407.2 (Pin_2), J408.2 (Pin_2), J409.2 (Pin_2), J410.2 (Pin_2), J411.2 (Pin_2), J412.2 (Pin_2), J413.3 (Pin_3), J414.3 (Pin_3), J415.35 (Pin_35), J415.36 (Pin_36), J416.2 (Pin_2), J417.3 (Pin_3), R407.1, R408.1, SW401.2, SWD401.1 (3V3), SWD401.2 (3V3)
- new net A0: J405.3 (Pin_3)
- new net A1: J405.4 (Pin_4)
- new net BOOT0: R406.1, SW401.1
- new net D0: J409.3 (Pin_3)
- new net D1: J409.4 (Pin_4)
- new net D4: J411.3 (Pin_3)
- new net D5: J411.4 (Pin_4)
- new net DBG_UART_RX: SWD401.4 (UART_RX)
- new net DBG_UART_TX: SWD401.6 (UART_TX)
- new net I2C2_SCL: J412.3 (Pin_3)
- new net I2C2_SDA: J412.4 (Pin_4)
- new net I2C5_SCL: J406.3 (Pin_3), J410.3 (Pin_3)
- new net I2C5_SDA: J406.4 (Pin_4), J410.4 (Pin_4)
- new net NRST: C401.1, SW402.1
- new net PA05: J413.8 (Pin_8)
- new net PA06: J413.6 (Pin_6)
- new net PA07: J413.4 (Pin_4)
- new net PB00: J415.29 (Pin_29)
- new net PB01: J415.30 (Pin_30)
- new net PB02: J415.27 (Pin_27)
- new net PC04: J413.2 (Pin_2)
- new net PC05: J413.5 (Pin_5)
- new net PD10: J415.14 (Pin_14)
- new net PD11: J415.11 (Pin_11)
- new net PD12: J415.12 (Pin_12)
- new net PD13: J415.9 (Pin_9)
- new net PD14: J415.10 (Pin_10)
- new net PD15: J415.7 (Pin_7)
- new net PE07: J415.22 (Pin_22)
- new net PE08: J415.19 (Pin_19)
- new net PE09: J415.20 (Pin_20)
- new net PE10: J415.17 (Pin_17)
- new net PE11: J415.18 (Pin_18)
- new net PE12: J415.15 (Pin_15)
- new net PE13: J415.16 (Pin_16)
- new net PE14: J415.13 (Pin_13)
- new net PF11: J415.28 (Pin_28)
- new net PF13: J415.25 (Pin_25)
- new net PF14: J415.26 (Pin_26)
- new net PF15: J415.23 (Pin_23)
- new net PG00: J415.24 (Pin_24)
- new net PG01: J415.21 (Pin_21)
- new net PG02: J415.8 (Pin_8)
- new net PG03: J415.5 (Pin_5)
- new net PG04: J415.6 (Pin_6)
- new net PG05: J415.3 (Pin_3)
- new net PG06: J415.4 (Pin_4)
- new net PG07: J415.1 (Pin_1)
- new net PG08: J415.2 (Pin_2)
- new net SPI1_CS: J417.8 (Pin_8)
- new net SPI1_IRQ: J417.5 (Pin_5)
- new net SPI1_MISO: J417.4 (Pin_4)
- new net SPI1_MOSI: J417.6 (Pin_6)
- new net SPI1_SCLK: J417.2 (Pin_2)
- new net SPI2_CS: J414.8 (Pin_8)
- new net SPI2_IRQ: J414.5 (Pin_5)
- new net SPI2_MISO: J414.4 (Pin_4)
- new net SPI2_MOSI: J414.6 (Pin_6)
- new net SPI2_SCLK: J414.2 (Pin_2)
- new net SWCLK: SWD401.5 (SWCLK)
- new net SWDIO: SWD401.3 (SWDIO)
- new net UART10_RX: J416.4 (Pin_4)
- new net UART10_TX: J416.3 (Pin_3)
- new net UART2_RX: J407.4 (Pin_4)
- new net UART2_TX: J407.3 (Pin_3)
- new net UART3_RX: J408.4 (Pin_4)
- new net UART3_TX: J408.3 (Pin_3)
- new net USR_BTN1: C402.1, R407.2, SW403.1
- new net USR_BTN2: C403.1, R408.2, SW404.1
- new net VBATT: J402.3 (Pin_3)
- no-connect marks 1 -> 3
Other:
- note added: "<- Facing"
- note added: "NOTE: I2C2 has pull ups I2C5 is without pull ups"
- note added: "ONLY USING 02X04"
- note removed: "B to A"
- note removed: "DIR: H:A->B L:B->A"
- company: (none) -> Scott CJX
- title: (none) -> Bigger Brain

Commit message: freeze rev1.1
Parts:
- added R409: 10k, Resistor_SMD:R_0603_1608Metric, symbol Device:R
- J402: Element14 (none) -> 1012243
- J403, J404, J405, J406, J407, J408, J409, J410, J411, J412, J416: Element14 (none) -> 9492496
- J413, J414, J417: Element14 (none) -> 1830787
Connections:
- net +3V3: now also R409.1
- net NRST: now also R409.2

Commit message: updated rev2
Parts:
- removed J403, J404, J405, J406, J407, J408, J409, J410, J411, J412, J416: PH_01x05V-H, NVF-Kicad:PH_01x05V-H, symbol Connector_Generic:Conn_01x05
- removed J413, J414, J417: PHD_02x04V-H, NVF-Kicad:PHD_02x04V-H, symbol Connector_Generic:Conn_02x04_Odd_Even
- removed SWD401: ~, NVF-Kicad:2.54mm2x04V-H, symbol NVF-Kicad:SWD_Breakout
- added D403: GREEN, LED_SMD:LED_0603_1608Metric, symbol Device:LED
- added D404: RED, LED_SMD:LED_0603_1608Metric, symbol Device:LED
- added D405, D406: BLUE, LED_SMD:LED_0603_1608Metric, symbol Device:LED
- added J404, J405, J406, J410, J411, J412: Conn_01x02, Connector_JST:JST_PH_B2B-PH-K_1x02_P2.00mm_Vertical, symbol Connector_Generic:Conn_01x02
- added J407, J408, J409: I2C Breakout, NVF-Kicad:PH_01x05V-H, symbol NVF_OwnParts:NVF-I2C-01x05
- added J413, J415, J416, J417, J418, J419, J422: Generic Breakout, NVF-Kicad:PH_01x05V-H, symbol NVF_OwnParts:NVF-AB-01x05
- added J414, J423, J424: UART Breakout, NVF-Kicad:PH_01x05V-H, symbol NVF_OwnParts:NVF-UART-01x05
- added J420, J421, J427: SPI Breakout, NVF-Kicad:PHD_02x04V-H, symbol NVF_OwnParts:NVF-SPI-02x04
- added J425, J426: Generic Breakout, NVF-Kicad:PH_01x05V-H, symbol NVF_OwnParts:NVF-I2C-01x05
- added R410, R411, R414: 1k, Resistor_SMD:R_0603_1608Metric, symbol Device:R
- added R412, R413: 200, Resistor_SMD:R_0603_1608Metric, symbol Device:R
- added SWD401: ~, NVF-Kicad:PHD_02x04V-H, symbol NVF_OwnParts:NVF-SWD-02x04/05
- R409: value 10k -> 200; LCSC C25804 -> C8218
- renumbered J415 to J403
Connections:
- net +3V3: now also D404.2 (A), D405.2 (A), SWD401.1 (3V3), SWD401.2 (3V3); no longer R409.1
- net +5V: now also D403.2 (A), J407.1 (5V), J408.1 (5V), J409.1 (5V), J413.1 (5V), J414.1 (5V), J415.1 (5V), J416.1 (5V), J417.1 (5V), J418.1 (5V), J419.1 (5V), J420.1 (5V), J421.1 (5V), J422.1 (5V), J423.1 (5V), J424.1 (5V), J425.1 (5V), J426.1 (5V), J427.1 (5V)
- net A0: now also J422.3 (A)
- net A1: now also J422.4 (B)
- net CAN1_H: now also J405.2 (Pin_2), J411.2 (Pin_2)
- net CAN1_L: now also J405.1 (Pin_1), J411.1 (Pin_1)
- net CAN2_H: now also J404.2 (Pin_2), J410.2 (Pin_2)
- net CAN2_L: now also J404.1 (Pin_1), J410.1 (Pin_1)
- net CAN3_H: now also J406.2 (Pin_2), J412.2 (Pin_2)
- net CAN3_L: now also J406.1 (Pin_1), J412.1 (Pin_1)
- net DBG_UART_RX: now also SWD401.4 (UART_RX)
- net DBG_UART_TX: now also SWD401.6 (UART_TX)
- net GND: now also R409.2, J407.5 (GND), J408.5 (GND), J409.5 (GND), J413.5 (GND), J414.5 (GND), J415.5 (GND), J416.5 (GND), J417.5 (GND), J418.5 (GND), J419.5 (GND), J420.8 (GND), J421.8 (GND), J422.5 (GND), J423.5 (GND), J424.5 (GND), J425.5 (GND), J426.5 (GND), J427.8 (GND), R412.2, R414.2, SWD401.7 (GND), SWD401.8 (GND)
- net I2C2_SCL: now also J425.3 (I2C_SCL), J426.3 (I2C_SCL)
- net I2C2_SDA: now also J425.4 (I2C_SDA), J426.4 (I2C_SDA)
- net I2C5_SCL: now also J407.3 (I2C_SCL), J408.3 (I2C_SCL), J409.3 (I2C_SCL)
- net I2C5_SDA: now also J407.4 (I2C_SDA), J408.4 (I2C_SDA), J409.4 (I2C_SDA)
- net NRST: no longer R409.2
- net PA05: now also J421.7 (CS)
- net PA06: now also J421.6 (MOSI)
- net PA07: now also J421.4 (MISO)
- net PC04: now also J421.2 (SCLK)
- net PC05: now also J421.5 (IRQ)
- net PWM1: now also J413.3 (A)
- net PWM2: now also J413.4 (B)
- net PWM3: now also J415.4 (B), J416.4 (B)
- net PWM4: now also J415.3 (A), J416.3 (A)
- net SPI1_CS: now also J420.7 (CS)
- net SPI1_IRQ: now also J420.5 (IRQ)
- net SPI1_MISO: now also J420.4 (MISO)
- net SPI1_MOSI: now also J420.6 (MOSI)
- net SPI1_SCLK: now also J420.2 (SCLK)
- net SPI2_CS: now also J427.7 (CS)
- net SPI2_IRQ: now also J427.5 (IRQ)
- net SPI2_MISO: now also J427.4 (MISO)
- net SPI2_MOSI: now also J427.6 (MOSI)
- net SPI2_SCLK: now also J427.2 (SCLK)
- net SWCLK: now also SWD401.5 (SWCLK)
- net SWDIO: now also SWD401.3 (SWDIO)
- net UART10_RX: now also J414.4 (UART_RX)
- net UART10_TX: now also J414.3 (UART_TX)
- net UART2_RX: now also J423.4 (UART_RX)
- net UART2_TX: now also J423.3 (UART_TX)
- net UART3_RX: now also J424.4 (UART_RX)
- net UART3_TX: now also J424.3 (UART_TX)
- net USR_BTN1: now also R410.1; no longer SW403.1
- net USR_BTN2: now also R411.1; no longer SW404.1
- net VCC: now also D406.2 (A)
- new net: D403.1 (K), R409.1
- new net: D405.1 (K), R413.1
- new net: D404.1 (K), R412.1
- new net: R410.2, SW403.1
- new net: D406.1 (K), R414.1
- new net: R411.2, SW404.1
- new net +3.3V: J407.2 (3V3), J408.2 (3V3), J409.2 (3V3), J413.2 (3V3), J414.2 (3V3), J415.2 (3V3), J416.2 (3V3), J417.2 (3V3), J418.2 (3V3), J419.2 (3V3), J420.3 (3V3), J421.3 (3V3), J422.2 (3V3), J423.2 (3V3), J424.2 (3V3), J425.2 (3V3), J426.2 (3V3), J427.3 (3V3)
- new net PB03: J417.3 (A)
- new net PB04: J417.4 (B)
- new net PE00: J418.3 (A)
- new net PE01: J418.4 (B)
- new net PG12: J419.3 (A)
- new net PG13: J419.4 (B)
- new net USR_LED: R413.2
Other:
- note added: "Assuming conditions: LED: V_{F}: 2.5V, I_{F}: 4mA Calculations for CLR: 3v3-2v5=0v8 V=IR: 0v8 = 0.04R R = 200"
- note added: "RCC"
- note added: "Ref: CLR Calculator"
- note added: "Ref: STM32 Pin Current MAX MCU MAX I_{IO(PIN)} = 25mA,"
- note added: "User Btn"
- moved on the sheet: C401, C402, C403, D401, D402, H401, H402, H403, H404, J402, J403, R403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

Commit message: freeze rev2
Parts:
- C401, C402, C403, D401, D402, D403, D404, D405, D406, H401, H402, H403, H404, J401, J403, R401, R402, R403, R404, R405, R406, R407, R408, R409, R410, R411, R412, R413, R414, SW401, SW402, SW403, SW404: Element14 (none) -> -
- J404, J405, J406, J410, J411, J412: Element14 (none) -> -; LCSC (none) -> -
- J407, J408, J409, J413, J414, J415, J416, J417, J418, J419, J422, J423, J424, J425, J426: Element14 (none) -> 9492445; LCSC (none) -> -
- J420, J421, J427, SWD401: Element14 (none) -> 1830787; LCSC (none) -> -

Commit message: updated rev2.1
Parts:
- added JP401: Jumper_2_Open, Connector_PinHeader_2.54mm:PinHeader_1x02_P2.54mm_Vertical, symbol Jumper:Jumper_2_Open
- C401, C402, C403, D401, D402, D403, D404, D405, D406, H401, H402, H403, H404, J401, R401, R402, R403, R404, R405, R406, R407, R408, R410, R411, R414, SW401, SW402, SW403, SW404: Assemble (none) -> 1
- J402: Assemble (none) -> 1; LCSC - -> C485575
- J403: Assemble (none) -> 0; LCSC - -> C2894981
- J404, J405, J406, J410, J411, J412: Assemble (none) -> 0; LCSC - -> C2683610
- J407, J408, J409, J413, J414, J415, J416, J417, J418, J419, J422, J423, J424, J425, J426: Assemble (none) -> 0; LCSC - -> C157993
- J420, J421, J427: Assemble (none) -> 0; LCSC - -> C157975
- R409, R412, R413: value 200 -> 300; Assemble (none) -> 1; LCSC C8218 -> C23025
- SWD401: Assemble (none) -> 1; LCSC - -> C157975
Connections:
- net +5V: now also JP401.2 (B)
- net VBUS: now also JP401.1 (A)
Other:
- moved on the sheet: D401, D402

Commit message: added fab and ibom
Parts:
- J404, J405, J406, J410, J411, J412: footprint Connector_JST:JST_PH_B2B-PH-K_1x02_P2.00mm_Vertical -> NVF-Kicad:PH_01x02V-H
Changed lines of the file:
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@@
 			)
 		)
-		(property "Footprint" "Connector_JST:JST_PH_B2B-PH-K_1x02_P2.00mm_Vertical"
+		(property "Footprint" "NVF-Kicad:PH_01x02V-H"
 			(at 137.16 111.76 0)
 			(effects
@@
 			)
 		)
-		(property "Footprint" "Connector_JST:JST_PH_B2B-PH-K_1x02_P2.00mm_Vertical"
+		(property "Footprint" "NVF-Kicad:PH_01x02V-H"
 			(at 137.16 101.6 0)
 			(effects
@@
 			)
 		)
-		(property "Footprint" "Connector_JST:JST_PH_B2B-PH-K_1x02_P2.00mm_Vertical"
+		(property "Footprint" "NVF-Kicad:PH_01x02V-H"
 			(at 104.14 101.6 0)
 			(effects
@@
 			)
 		)
-		(property "Footprint" "Connector_JST:JST_PH_B2B-PH-K_1x02_P2.00mm_Vertical"
+		(property "Footprint" "NVF-Kicad:PH_01x02V-H"
 			(at 104.14 111.76 0)
 			(effects
@@
 			)
 		)
-		(property "Footprint" "Connector_JST:JST_PH_B2B-PH-K_1x02_P2.00mm_Vertical"
+		(property "Footprint" "NVF-Kicad:PH_01x02V-H"
 			(at 120.65 111.76 0)
 			(effects
@@
 			)
 		)
-		(property "Footprint" "Connector_JST:JST_PH_B2B-PH-K_1x02_P2.00mm_Vertical"
+		(property "Footprint" "NVF-Kicad:PH_01x02V-H"
 			(at 120.65 101.6 0)
 			(effects
