File: HDK/Power.kicad_sch (KiCad schematic)
At the start: 34 parts, among them U201 AMS1117-3.3, U202 AMS1117-3.3, U203 AMS1117-3.3

Commit message: updated WIP
Parts:
- added D202, D203: D, symbol Device:D
- C225, C226: renamed from C113; now not fitted; now left out of the parts list
- U202: now not fitted; now left out of the parts list
- renumbered C101 to C201, C102 to C202, C103 to C203, C104 to C204, C105 to C205, C106 to C206, C107 to C207, C108 to C208, C109 to C209, C110 to C210, C111 to C211, C112 to C212, C113 to C213, C114 to C214, C115 to C215, C116 to C216, C117 to C217, C118 to C218, C119 to C219, C120 to C220, C121 to C221, C122 to C222, C113 to C223, C113 to C224, C113 to C227, C113 to C228, D101 to D201, L101 to L201, R101 to R201
Connections:
- net VCC: now also D202.1 (K), D203.1 (K)
- new net V1: D202.2 (A)
- new net V2: D203.2 (A)

Commit message: added rev1-final
Parts:
- removed D202, D203: D, symbol Device:D
- added D401 (x2): SS14, Diode_SMD:D_SMA, symbol Device:D_Schottky
- added F201, F202: 1A, NVF-Kicad:FUSE-MCCQ-122, symbol Device:Fuse
- added R202, R204: 5k1, Resistor_SMD:R_0603_1608Metric, symbol Device:R
- added R203, R205: 1k, Resistor_SMD:R_0603_1608Metric, symbol Device:R
- C201, C202, C203, C204, C205, C206, C207, C208, C209, C210, C211, C213, C215, C217, C221: LCSC C57112 -> C14663
- U203: value AMS1117-3.3 -> AMS1117-5.0
Connections:
- net GND: now also R203.2, R205.2
- net V1: now also F201.1
- net V2: now also F202.1
- net VCC: now also D401.1 (K), D401.1 (K)
- new net V1_F: D401.2 (A), F201.2, R202.2
- new net V1_SENSE: R202.1, R205.1
- new net V2_F: D401.2 (A), F202.2, R204.2
- new net V2_SENSE: R203.1, R204.1
Other:
- company: (none) -> Scott CJX
- title: (none) -> Bigger Brain

Commit message: fixed bom
Parts:
- U202: LCSC C6186 -> -
- U203: LCSC C6186 -> C6187
Changed lines of the file:
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@@
       (effects (font (size 1.27 1.27)) hide)
     )
-    (property "LCSC" "C6186" (at 82.55 151.13 0)
+    (property "LCSC" "-" (at 82.55 151.13 0)
       (effects (font (size 1.27 1.27)) hide)
     )
@@
       (effects (font (size 1.27 1.27)) hide)
     )
-    (property "LCSC" "C6186" (at 125.73 151.13 0)
-      (effects (font (size 1.27 1.27)) hide)
-    )
+    (property "LCSC" "C6187" (at 125.73 151.13 0)
+      (effects (font (size 1.27 1.27)) hide)
+    )
