File: HDK/Power.kicad_sch (KiCad schematic)
At the start: 42 parts, among them U201 AMS1117-3.3, U202 AMS1117-3.3, U203 AMS1117-5.0

Commit message: updated rev2
Parts:
- F201, F202: footprint NVF-Kicad:FUSE-MCCQ-122 -> NVF-Kicad:FUSE-Littelfuse_Nano2_154x
Connections:
- net +3V3 is gone; now on net +3.3V: C201.1, C202.1, C203.1, C204.1, C205.1, C206.1, C207.1, C208.1, C209.1, C210.1, C211.1, C212.1, C213.1, C214.1, C224.1, D201.1 (A), L201.1, U201.2 (VO)
Changed lines of the file:
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@@
 	(title_block
 		(title "Bigger Brain")
-		(date "2024-02-21")
-		(rev "1.1")
+		(date "2024-03-05")
+		(rev "2")
 		(company "Scott CJX")
 	)
@@
 	(wire
 		(pts
+			(xy 31.75 186.69) (xy 39.37 186.69)
+		)
+		(stroke
+			(width 0)
+			(type default)
+		)
+	)
+	(wire
+		(pts
 			(xy 124.46 177.8) (xy 134.62 177.8)
 		)
@@
 		)
 	)
+	(global_label "MCU-3.3V"
+		(shape input)
+		(at 39.37 186.69 0)
+		(fields_autoplaced yes)
+		(effects
+			(font
+				(size 1.27 1.27)
+			)
+			(justify left)
+		)
+		(property "Intersheetrefs" "${INTERSHEET_REFS}"
+			(at 52.0919 186.69 0)
+			(effects
+				(font
+					(size 1.27 1.27)
+				)
+				(justify left)
+				(hide yes)
+			)
+		)
+	)
 	(global_label "V1"
 		(shape input)
@@
 		)
 	)
+	(global_label "PP-3.3V"
+		(shape input)
+		(at 31.75 186.69 180)
+		(fields_autoplaced yes)
+		(effects
+			(font
+				(size 1.27 1.27)
+			)
+			(justify right)
+		)
+		(property "Intersheetrefs" "${INTERSHEET_REFS}"
+			(at 20.54 186.69 0)
+			(effects
+				(font
+					(size 1.27 1.27)
+				)
+				(justify right)
+				(hide yes)
+			)
+		)
+	)
 	(global_label "V2"
 		(shape input)
@@
 			)
 		)
-		(property "Footprint" "NVF-Kicad:FUSE-MCCQ-122"
+		(property "Footprint" "NVF-Kicad:FUSE-Littelfuse_Nano2_154x"
 			(at 68.58 179.578 90)
 			(effects
@@
 			)
 		)
-		(property "Footprint" "NVF-Kicad:FUSE-MCCQ-122"
+		(property "Footprint" "NVF-Kicad:FUSE-Littelfuse_Nano2_154x"
 			(at 68.58 184.658 90)
 			(effects

Commit message: freeze rev2
Parts:
- C201, C202, C203, C204, C205, C206, C207, C208, C209, C210, C211, C212, C213, C214, C215, C216, C217, C218, C219, C220, C221, C222, C223, C224, C225, C226, C227, C228, D201, D202, D203, L201, R201, R202, R203, R204, R205, U201, U202, U203: Element14 (none) -> -
Changed lines of the file:
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@@
 			)
 		)
-		(property "Element14" ""
+		(property "Element14" "-"
 			(at 35.56 34.29 0)
 			(effects
@@
 			)
 		)
-		(property "Element14" ""
+		(property "Element14" "-"
 			(at 88.9 182.88 0)
 			(effects
@@
 			)
 		)
-		(property "Element14" ""
+		(property "Element14" "-"
 			(at 88.9 177.8 0)
 			(effects
@@
 			)
 		)
-		(property "Element14" ""
+		(property "Element14" "-"
 			(at 46.99 52.07 0)
 			(effects
@@
 			)
 		)
-		(property "Element14" ""
+		(property "Element14" "-"
 			(at 39.37 151.13 0)
 			(effects
@@
 			)
 		)
-		(property "Element14" ""
+		(property "Element14" "-"
 			(at 53.34 156.21 0)
 			(effects
@@
 			)
 		)
-		(property "Element14" ""
+		(property "Element14" "-"
 			(at 24.13 34.29 0)
 			(effects
@@
 			)
 		)
-		(property "Element14" ""
+		(property "Element14" "-"
 			(at 58.42 34.29 0)
 			(effects
@@
 			)
 		)
-		(property "Element14" ""
+		(property "Element14" "-"
 			(at 96.52 52.07 0)
 			(effects
@@
 			)
 		)
-		(property "Element14" ""
+		(property "Element14" "-"
 			(at 31.75 120.65 0)
 			(effects
@@
 			)
 		)
-		(property "Element14" ""
+		(property "Element14" "-"
 			(at 82.55 151.13 0)
 			(effects
@@
 			)
 		)
-		(property "Element14" ""
+		(property "Element14" "-"
 			(at 135.89 87.63 0)
 			(effects
@@
 			)
 		)
-		(property "Element14" ""
+		(property "Element14" "-"
 			(at 69.85 52.07 0)
 			(effects
@@
 			)
 		)
-		(property "Element14" ""
+		(property "Element14" "-"
 			(at 113.03 177.8 0)
 			(effects
@@
 			)
 		)
-		(property "Element14" ""
+		(property "Element14" "-"
 			(at 46.99 34.29 0)
 			(effects
@@
 			)
 		)
-		(property "Element14" ""
+		(property "Element14" "-"
 			(at 119.38 187.96 0)
 			(effects
@@
 			)
 		)
-		(property "Element14" ""
+		(property "Element14" "-"
 			(at 124.46 187.96 0)
 			(effects
@@
 			)
 		)
-		(property "Element14" ""
+		(property "Element14" "-"
 			(at 113.03 182.88 0)
 			(effects
@@
 			)
 		)
-		(property "Element14" ""
+		(property "Element14" "-"
 			(at 69.85 34.29 0)
 			(effects
@@
 			)
 		)
-		(property "Element14" ""
+		(property "Element14" "-"
 			(at 25.4 156.21 0)
 			(effects
@@
 			)
 		)
-		(property "Element14" ""
+		(property "Element14" "-"
 			(at 68.58 156.21 0)
 			(effects
@@
 			)
 		)
-		(property "Element14" ""
+		(property "Element14" "-"
 			(at 24.13 52.07 0)
 			(effects
@@
 			)
 		)
-		(property "Element14" ""
+		(property "Element14" "-"
 			(at 125.73 151.13 0)
 			(effects
@@
 			)
 		)
-		(property "Element14" ""
+		(property "Element14" "-"
 			(at 58.42 52.07 0)
 			(effects
@@
 			)
 		)
-		(property "Element14" ""
+		(property "Element14" "-"
 			(at 124.46 121.92 0)
 			(effects
@@
 			)
 		)
-		(property "Element14" ""
+		(property "Element14" "-"
 			(at 81.28 52.07 0)
 			(effects
@@
 			)
 		)
-		(property "Element14" ""
+		(property "Element14" "-"
 			(at 71.12 86.36 0)
 			(effects
@@
 			)
 		)
-		(property "Element14" ""
+		(property "Element14" "-"
 			(at 39.37 87.63 0)
 			(effects
@@
 			)
 		)
-		(property "Element14" ""
+		(property "Element14" "-"
 			(at 107.95 116.84 0)
 			(effects
@@
 			)
 		)
-		(property "Element14" ""
+		(property "Element14" "-"
 			(at 124.46 87.63 0)
 			(effects
@@
 			)
 		)
-		(property "Element14" ""
+		(property "Element14" "-"
 			(at 44.45 120.65 0)
 			(effects
@@
 			)
 		)
-		(property "Element14" ""
+		(property "Element14" "-"
 			(at 107.95 52.07 0)
 			(effects
@@
 			)
 		)
-		(property "Element14" ""
+		(property "Element14" "-"
 			(at 107.95 82.55 0)
 			(effects
@@
 			)
 		)
-		(property "Element14" ""
+		(property "Element14" "-"
 			(at 59.69 86.36 0)
 			(effects
@@
 			)
 		)
-		(property "Element14" ""
+		(property "Element14" "-"
 			(at 35.56 52.07 0)
 			(effects
@@
 			)
 		)
-		(property "Element14" ""
+		(property "Element14" "-"
 			(at 135.89 121.92 0)
 			(effects
@@
 			)
 		)
-		(property "Element14" ""
+		(property "Element14" "-"
 			(at 111.76 156.21 0)
 			(effects
@@
 			)
 		)
-		(property "Element14" ""
+		(property "Element14" "-"
 			(at 96.52 156.21 0)
 			(effects
@@
 			)
 		)
-		(property "Element14" ""
+		(property "Element14" "-"
 			(at 139.7 156.21 0)
 			(effects
@@
 			)
 		)
-		(property "Element14" ""
+		(property "Element14" "-"
 			(at 81.28 34.29 0)
 			(effects
