File: HDK/Power.kicad_sch (KiCad schematic)
At the start: 42 parts, among them U201 AMS1117-3.3, U202 AMS1117-3.3, U203 AMS1117-5.0

Commit message: freeze rev2
Parts:
- L201: LCSC GZ2012D101TF -> C1015
- U203: LCSC C6186 -> C6187
Changed lines of the file:
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@@
 			)
 		)
-		(property "LCSC" "C6186"
+		(property "LCSC" "C6187"
 			(at 125.73 151.13 0)
 			(effects
@@
 			)
 		)
-		(property "LCSC" "GZ2012D101TF"
+		(property "LCSC" "C1015"
 			(at 107.95 82.55 0)
 			(effects

Commit message: updated rev2.1
Parts:
- C201, C202, C203, C204, C205, C206, C207, C208, C209, C210, C211, C212, C213, C214, C215, C216, C217, C218, C219, C220, C221, C222, C223, C224, C227, C228, D201, D202, D203, L201, R201, R202, R203, R204, R205, U201, U203: Assemble (none) -> 1
- F201, F202: Assemble (none) -> 1; LCSC - -> C206910
