File: HDK/bigger-brain.kicad_pcb (KiCad board)
At the start: 4 copper layers, 100 x 100 mm, 78 parts, among them J301 Micro_SD_Card_Det1, J401 USB_C_Receptacle_USB2.0, J402 Conn_02x12_Top_Bottom, U101 STM32H723ZGTx, U201 AMS1117-3.3, U202 AMS1117-3.3, U203 AMS1117-3.3, U401 74HC245, U501 TJA1042T-3, U601 TJA1042T-3, U701 TJA1042T-3, X101 25MHz ±10ppm, Y101 32.768kHz 12.5pF ±20ppm

Commit message: updated WIP
Parts:
- removed C225, C226: 2u2, Capacitor_SMD:C_0805_2012Metric
- removed the REF** at (70.2, 136.8)
- removed the REF** at (70.2, 129.3)
- removed the REF** at (70.2, 144.5)
- removed the REF** at (84.7, 136.6)
- removed the REF** at (84.7, 144.3)
- removed the REF** at (84.7, 129.2)
- removed U202: AMS1117-3.3, Package_TO_SOT_SMD:SOT-223-3_TabPin2
- added REF**: MountingHole_4.3mm_M4_DIN965_Pad_TopBottom, MountingHole:MountingHole_4.3mm_M4_DIN965_Pad_TopBottom, F.Cu at (144.0, 144.0)
- added REF**: MountingHole_4.3mm_M4_DIN965_Pad_TopBottom, MountingHole:MountingHole_4.3mm_M4_DIN965_Pad_TopBottom, F.Cu at (56.0, 56.0)
- added REF**: MountingHole_4.3mm_M4_DIN965_Pad_TopBottom, MountingHole:MountingHole_4.3mm_M4_DIN965_Pad_TopBottom, F.Cu at (144.0, 56.0)
- J402: footprint Connector_Molex:Molex_Mini-Fit_Jr_5566-24A_2x12_P4.20mm_Vertical -> NVF-Kicad-Resources:Micro-Fit_2x12V-H
- moved C401 103.7 mm to (80.1, 70.5)
- moved U201 65.8 mm to (76.1, 126.1), turned to 0 degrees
- moved U203 65.5 mm to (76.1, 118.1), turned to 0 degrees
- moved C223 65.1 mm to (69.7, 128.4)
- moved C224 65.0 mm to (69.7, 126.1)
- moved C227 64.8 mm to (69.8, 120.4)
- moved C228 64.7 mm to (69.8, 118.1)
- moved kibuzzard-65AE28D0 58.0 mm to (136.5, 113.2)
- moved R401 49.0 mm to (143.2, 106.7), turned to 180 degrees
- moved R402 48.6 mm to (143.2, 108.6), turned to 180 degrees
- moved U401 37.8 mm to (75.3, 74.8)
- moved C601 5.95 mm to (80.3, 85.0)
- moved C602 5.95 mm to (73.6, 81.3)
- moved R403 5.95 mm to (69.2, 84.2)
- moved R601 5.95 mm to (73.6, 88.8)
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Connections:
- U101 pad 122: /SD2_CLK -> unconnected-(U101-PD6-Pad122)
- U101 pad 123: /SD2_CMD -> unconnected-(U101-PD7-Pad123)
- U101 pad 124: /SD2_DAT0 -> unconnected-(U101-PG9-Pad124)
- U101 pad 125: /SD2_DAT1 -> unconnected-(U101-PG10-Pad125)
- U101 pad 126: /SD2_DAT2 -> unconnected-(U101-PG11-Pad126)
- U101 pad 127: /SD2_DAT3 -> unconnected-(U101-PG12-Pad127)
- U401 pad 7: unconnected-(U401-A5-Pad7) -> /HMI/DET3_A
- U401 pad 8: unconnected-(U401-A6-Pad8) -> /HMI/DET1_A
- U401 pad 9: unconnected-(U401-A7-Pad9) -> /HMI/DET2_A
Routing:
- net V1: track 0.00 -> 47.3 mm
- net /HMI/DET2_A: track 0.00 -> 45.7 mm, vias 0 -> 1
- net /HMI/DET1_A: track 0.00 -> 34.8 mm, vias 0 -> 1
- net V2: track 0.00 -> 32.6 mm
- net /HMI/DET3_A: track 0.00 -> 23.9 mm, vias 0 -> 1
- net /HMI/CC2: track 0.00 -> 14.0 mm
- net /HMI/CC1: track 0.00 -> 9.10 mm
- net GND: track 49.5 -> 58.0 mm, vias 57 -> 66
- net /HMI/DET3_B: track 0.00 -> 8.42 mm, vias 0 -> 1
- net /HMI/DET1_B: track 0.00 -> 8.42 mm, vias 0 -> 1
- net /CAN2_RX: track 36.6 -> 32.7 mm
- net PP-5.0V: track 11.0 -> 14.7 mm, vias 3 -> 4
- net /CAN3_TX: track 29.3 -> 26.1 mm
- net /HMI/CAN2_L-T: track 17.2 -> 14.9 mm
- net /HMI/CAN3_L-T: track 16.8 -> 14.6 mm
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- added copper zone on F.Cu, net MCU-3.3V
- added copper zone on F.Cu, net PP-5.0V
- added copper zone on F.Cu, net VCC
Other:
- board text added: "JLCJLCJLCJLC"

Commit message: added rev1-final
Parts:
- removed R501, R601, R701: 10k, Resistor_SMD:R_0603_1608Metric
- removed U401: 74HC245, Package_SO:TSSOP-20_4.4x6.5mm_P0.65mm
- added C402: 100n, Capacitor_SMD:C_0603_1608Metric, F.Cu at (118.0, 84.8)
- added C403: 100n, Capacitor_SMD:C_0603_1608Metric, F.Cu at (126.4, 84.8)
- added D202: SS14, Diode_SMD:D_SMA, F.Cu at (69.4, 159.1)
- added D203: SS14, Diode_SMD:D_SMA, F.Cu at (69.4, 163.6)
- added D401: SS14, Diode_SMD:D_SMA, F.Cu at (143.7, 138.8)
- added D402: SS14, Diode_SMD:D_SMA, F.Cu at (139.7, 138.8)
- added F201: 1A, NVF-Kicad:FUSE-MCCQ-122, F.Cu at (61.8, 154.1)
- added F202: 1A, NVF-Kicad:FUSE-MCCQ-122, F.Cu at (55.8, 154.1)
- added G***: LOGO, NVF-Kicad:NVF-Logo-30mm, F.Cu at (136.8, 157.4)
- added G***: LOGO, NVF-Kicad:NVF-Logo-30mm, B.Cu at (109.9, 113.4)
- added J403: PH_01x05V-H, NVF-Kicad:PH_01x05V-H, F.Cu at (71.2, 82.0)
- added J404: PH_01x05V-H, NVF-Kicad:PH_01x05V-H, F.Cu at (89.2, 96.0)
- added J405: PH_01x05V-H, NVF-Kicad:PH_01x05V-H, F.Cu at (71.2, 96.0)
- added J406: PH_01x05V-H, NVF-Kicad:PH_01x05V-H, F.Cu at (80.2, 82.0)
- added J407: PH_01x05V-H, NVF-Kicad:PH_01x05V-H, F.Cu at (83.6, 153.9)
- added J408: PH_01x05V-H, NVF-Kicad:PH_01x05V-H, F.Cu at (110.6, 153.9)
- added J409: PH_01x05V-H, NVF-Kicad:PH_01x05V-H, F.Cu at (98.2, 96.0)
- added J410: PH_01x05V-H, NVF-Kicad:PH_01x05V-H, F.Cu at (89.2, 82.0)
- added J411: PH_01x05V-H, NVF-Kicad:PH_01x05V-H, F.Cu at (98.2, 82.0)
- added J412: PH_01x05V-H, NVF-Kicad:PH_01x05V-H, F.Cu at (101.6, 153.9)
- added J413: PHD_02x04V-H, NVF-Kicad:PHD_02x04V-H, F.Cu at (92.6, 153.9)
- added J414: PHD_02x04V-H, NVF-Kicad:PHD_02x04V-H, F.Cu at (119.6, 153.9)
- added J415: 2.54mm2x20V-H, NVF-Kicad:2.54mm2x20V-H, F.Cu at (107.4, 167.2)
- added J416: PH_01x05V-H, NVF-Kicad:PH_01x05V-H, F.Cu at (80.2, 96.0)
- added J417: PHD_02x04V-H, NVF-Kicad:PHD_02x04V-H, F.Cu at (107.2, 82.0)
- added R101: 5k1, Resistor_SMD:R_0603_1608Metric, F.Cu at (97.5, 153.8)
- added R102: 5k1, Resistor_SMD:R_0603_1608Metric, F.Cu at (97.5, 156.3)
- added R202: 5k1, Resistor_SMD:R_0603_1608Metric, F.Cu at (68.2, 168.9)
- added R203: 1k, Resistor_SMD:R_0603_1608Metric, F.Cu at (72.2, 167.1)
- added R204: 5k1, Resistor_SMD:R_0603_1608Metric, F.Cu at (68.2, 167.1)
- added R205: 1k, Resistor_SMD:R_0603_1608Metric, F.Cu at (72.2, 168.9)
- added R406: 10k, Resistor_SMD:R_0603_1608Metric, F.Cu at (63.2, 89.5)
- added R407: 10k, Resistor_SMD:R_0603_1608Metric, F.Cu at (118.0, 88.0)
- added R408: 10k, Resistor_SMD:R_0603_1608Metric, F.Cu at (126.4, 88.0)
- added SW401: SW_Push, NVF-Kicad:PushBtn_TS-1187A-B-A-B, F.Cu at (57.0, 91.4)
- added SW402: SW_Push, NVF-Kicad:PushBtn_TS-1187A-B-A-B, F.Cu at (57.0, 99.4)
- added SW403: SW_Push, NVF-Kicad:PushBtn_TS-1187A-B-A-B, F.Cu at (122.2, 82.6)
- added SW404: SW_Push, NVF-Kicad:PushBtn_TS-1187A-B-A-B, F.Cu at (130.6, 82.6)
- added SWD401: ~, NVF-Kicad:2.54mm2x04V-H, F.Cu at (142.4, 114.6)
- added kibuzzard-65BA50A4: G***, kibuzzard-65BA50A4, B.Cu at (118.8, 122.0)
- added kibuzzard-65BA50D8: G***, kibuzzard-65BA50D8, B.Cu at (106.4, 128.4)
- H401, H402, H403, H404: renamed from REF**; value MountingHole_4.3mm_M4_DIN965_Pad_TopBottom -> M4 Pad
- J301: value Micro_SD_Card_Det1 -> TF-01A; footprint NVF-Kicad:TF-01A -> NVF-Kicad:TFCard_TF-01A
- J401: value USB_C_Receptacle_USB2.0 -> USB_C; footprint NVF-Kicad:USB_C_Receptacle_HRO_TYPE-C-31-M-12 -> NVF-Kicad:USBC_HRO_TYPE-C-31-M-12
- J402: value Conn_02x12_Top_Bottom -> MicroFit_02x10V-H; footprint NVF-Kicad-Resources:Micro-Fit_2x12V-H -> NVF-Kicad:MicroFit_02x10V-H
- U203: value AMS1117-3.3 -> AMS1117-5.0
- moved kibuzzard-65AE28D0 34.0 mm to (136.5, 147.2)
- moved C401 31.8 mm to (63.2, 97.5)
- moved R403 28.6 mm to (69.2, 112.8)
- moved U601 28.6 mm to (75.2, 113.6)
- moved C601 28.5 mm to (80.3, 113.6)
- moved C602 28.5 mm to (73.6, 109.8)
- moved R404 25.6 mm to (69.2, 121.9)
- moved C502 25.5 mm to (73.5, 118.9)
- moved C501 25.5 mm to (80.0, 122.5)
- moved U501 25.5 mm to (75.2, 122.6)
- moved C201 25.4 mm to (93.2, 124.2)
- moved U201 25.3 mm to (74.6, 151.4)
- moved C223 25.3 mm to (68.2, 153.7)
- moved C224 25.3 mm to (68.2, 151.4)
- moved C227 25.3 mm to (68.2, 145.7)
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Connections:
- C401 pad 1: PP-5.0V -> NRST
- H401 pad 1: (no net) -> GND
- H402 pad 1: (no net) -> GND
- H403 pad 1: (no net) -> GND
- H404 pad 1: (no net) -> GND
- J402 pad 10: /CanTrx3/CAN_H -> V2
- J402 pad 11: /HMI/DET2_A -> /HMI/CAN2_L-T
- J402 pad 12: /HMI/DET2_B -> /CanTrx2/CAN_H
- J402 pad 13: /HMI/CAN2_L-T -> GND
- J402 pad 14: /CanTrx2/CAN_H -> /HMI/CAN1_L-T
- J402 pad 15: V1 -> /CanTrx1/CAN_H
- J402 pad 16: V1_A -> GND
- J402 pad 17: /HMI/CAN1_L-T -> /HMI/CAN3_L-T
- J402 pad 18: /CanTrx1/CAN_H -> /CanTrx3/CAN_H
- J402 pad 19: V2 -> GND
- J402 pad 20: V2_A -> GND
- J402 pad 3: /HMI/DET3_A -> VBATT
- J402 pad 4: /HMI/DET3_B -> /CanTrx1/CAN_L
- J402 pad 5: /CanTrx1/CAN_L -> /CanTrx1/CAN_H
- J402 pad 6: /CanTrx1/CAN_H -> GND
- J402 pad 7: /HMI/DET1_A -> /CanTrx3/CAN_L
- J402 pad 8: /HMI/DET1_B -> /CanTrx3/CAN_H
- J402 pad 9: /CanTrx3/CAN_L -> V1
- R306 pad 1: /SDCard1/SD_DET -> /SD1_DET
- U101 pad 1: unconnected-(U101-PE2-Pad1) -> /UART10_TX
- U101 pad 10: unconnected-(U101-PF0-Pad10) -> /I2C5_SDA
- U101 pad 101: unconnected-(U101-PA9-Pad101) -> /UART1_TX
- U101 pad 102: unconnected-(U101-PA10-Pad102) -> /UART1_RX
- U101 pad 11: unconnected-(U101-PF1-Pad11) -> /I2C5_SCL
- U101 pad 110: unconnected-(U101-PA15(JTDI)-Pad110) -> /SD1_DET
- U101 pad 114: unconnected-(U101-PD0-Pad114) -> USR_BTN2
- U101 pad 115: unconnected-(U101-PD1-Pad115) -> USR_BTN1
- U101 pad 12: unconnected-(U101-PF2-Pad12) -> PF02
- U101 pad 122: unconnected-(U101-PD6-Pad122) -> /SPI1_IRQ
- U101 pad 123: unconnected-(U101-PD7-Pad123) -> /SPI1_MOSI
- U101 pad 124: unconnected-(U101-PG9-Pad124) -> /SPI1_MISO
- U101 pad 125: unconnected-(U101-PG10-Pad125) -> /SPI1_CS
- U101 pad 126: unconnected-(U101-PG11-Pad126) -> /SPI1_SCLK
- U101 pad 13: unconnected-(U101-PF3-Pad13) -> PF03
- U101 pad 14: unconnected-(U101-PF4-Pad14) -> PF04
- U101 pad 141: unconnected-(U101-PE0-Pad141) -> PE00
- U101 pad 142: unconnected-(U101-PE1-Pad142) -> PE01
- U101 pad 15: unconnected-(U101-PF5-Pad15) -> PF05
- U101 pad 2: unconnected-(U101-PE3-Pad2) -> /UART10_RX
- U101 pad 3: unconnected-(U101-PE4-Pad3) -> PE04
- U101 pad 34: unconnected-(U101-PA0-Pad34) -> /V2_SENSE
- U101 pad 35: unconnected-(U101-PA1-Pad35) -> /V1_SENSE
- U101 pad 36: unconnected-(U101-PA2-Pad36) -> /UART2_TX
- U101 pad 37: unconnected-(U101-PA3-Pad37) -> /UART2_RX
- U101 pad 4: unconnected-(U101-PE5-Pad4) -> PE05
- U101 pad 41: unconnected-(U101-PA5-Pad41) -> PA05
- U101 pad 42: unconnected-(U101-PA6-Pad42) -> PA06
- U101 pad 43: unconnected-(U101-PA7-Pad43) -> PA07
- U101 pad 44: unconnected-(U101-PC4-Pad44) -> PC04
- U101 pad 45: unconnected-(U101-PC5-Pad45) -> PC05
- U101 pad 46: unconnected-(U101-PB0-Pad46) -> PB00
- U101 pad 47: unconnected-(U101-PB1-Pad47) -> PB01
- U101 pad 48: unconnected-(U101-PB2-Pad48) -> PB02
- U101 pad 49: unconnected-(U101-PF11-Pad49) -> PF11
- U101 pad 5: unconnected-(U101-PE6-Pad5) -> PE06
- U101 pad 53: unconnected-(U101-PF13-Pad53) -> PF13
- U101 pad 54: unconnected-(U101-PF14-Pad54) -> PF14
- U101 pad 55: unconnected-(U101-PF15-Pad55) -> PF15
- U101 pad 56: unconnected-(U101-PG0-Pad56) -> PG00
- U101 pad 57: unconnected-(U101-PG1-Pad57) -> PG01
- U101 pad 58: unconnected-(U101-PE7-Pad58) -> PE07
- U101 pad 59: unconnected-(U101-PE8-Pad59) -> PE08
- U101 pad 60: unconnected-(U101-PE9-Pad60) -> PE09
- U101 pad 63: unconnected-(U101-PE10-Pad63) -> PE10
- U101 pad 64: unconnected-(U101-PE11-Pad64) -> PE11
- U101 pad 65: unconnected-(U101-PE12-Pad65) -> PE12
- U101 pad 66: unconnected-(U101-PE13-Pad66) -> PE13
- U101 pad 67: unconnected-(U101-PE14-Pad67) -> PE14
- U101 pad 68: unconnected-(U101-PE15-Pad68) -> /SPI2_IRQ
- U101 pad 69: unconnected-(U101-PB10-Pad69) -> /I2C2_SCL
- U101 pad 70: unconnected-(U101-PB11-Pad70) -> /I2C2_SDA
- U101 pad 73: unconnected-(U101-PB12-Pad73) -> /SPI2_CS
- U101 pad 74: unconnected-(U101-PB13-Pad74) -> /SPI2_SCLK
- U101 pad 75: unconnected-(U101-PB14-Pad75) -> /SPI2_MISO
- U101 pad 76: unconnected-(U101-PB15-Pad76) -> /SPI2_MOSI
- U101 pad 77: unconnected-(U101-PD8-Pad77) -> /UART3_TX
- U101 pad 78: unconnected-(U101-PD9-Pad78) -> /UART3_RX
- U101 pad 79: unconnected-(U101-PD10-Pad79) -> PD10
- U101 pad 80: unconnected-(U101-PD11-Pad80) -> PD11
- U101 pad 81: unconnected-(U101-PD12-Pad81) -> PD12
- U101 pad 82: unconnected-(U101-PD13-Pad82) -> PD13
- U101 pad 85: unconnected-(U101-PD14-Pad85) -> PD14
- U101 pad 86: unconnected-(U101-PD15-Pad86) -> PD15
- U101 pad 87: unconnected-(U101-PG2-Pad87) -> PG02
- U101 pad 88: unconnected-(U101-PG3-Pad88) -> PG03
- U101 pad 89: unconnected-(U101-PG4-Pad89) -> PG04
- U101 pad 90: unconnected-(U101-PG5-Pad90) -> PG05
- U101 pad 91: unconnected-(U101-PG6-Pad91) -> PG06
- U101 pad 92: unconnected-(U101-PG7-Pad92) -> PG07
- U101 pad 93: unconnected-(U101-PG8-Pad93) -> PG08
- U501 pad 8: /CanTrx1/CAN_STB -> GND
- U601 pad 8: /CanTrx2/CAN_STB -> GND
- U701 pad 8: /CanTrx3/CAN_STB -> GND
Routing:
- net VCC: track 0.00 -> 130.3 mm, vias 0 -> 2
- net BOOT0: track 0.00 -> 69.8 mm, vias 0 -> 2
- net PF05: track 0.00 -> 69.7 mm, vias 0 -> 2
- net NRST: track 7.70 -> 73.6 mm, vias 1 -> 2
- net PF04: track 0.00 -> 65.3 mm, vias 0 -> 2
- net /I2C5_SCL: track 0.00 -> 62.8 mm, vias 0 -> 2
- net PG08: track 0.00 -> 60.3 mm
- net PG06: track 0.00 -> 59.1 mm
- net /I2C5_SDA: track 0.00 -> 58.9 mm, vias 0 -> 2
- net PG04: track 0.00 -> 57.9 mm
- net PG02: track 0.00 -> 56.8 mm
- net PG07: track 0.00 -> 56.7 mm
- net PD14: track 0.00 -> 55.5 mm
- net PG05: track 0.00 -> 55.5 mm
- net PE05: track 0.00 -> 54.8 mm
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Other:
- outline, holes or cut-outs redrawn
- board text added: "0.0000 mm / 0.0000 mm"
- board text added: "0.3000 mm"
- board text added: "01 02 03 04 05 06 07 08 09 10 11 12 12 14 15 16 17 18 19 20"
- board text added: "1.6000 mm"
- board text added: "100.0000 mm x 100.0000 mm"
- board text added: "3V3"
- board text added: "4"
- board text added: "5V"
- board text added: "ANA"
- board text added: "ANA/ SPI1"
- board text added: "ANA/ UART2"
- board text added: "BOARD CHARACTERISTICS"
- board text added: "BOOT0"
- board text added: "Bigger-Brain Rev1"
- board text added: "Board Thickness:"
- board text added: "Board overall dimensions:"
- board text added: "CAN1"
- board text added: "CAN2"
- board text added: "CAN3"
- board text added: "Castellated pads:"
- board text added: "Copper Finish:"
- board text added: "Copper Layer Count:"
- board text added: "Edge card connectors:"
- board text added: "G CLK DIO 3V3"
- board text added: "G TX RX 3V3"
- board text added: "I2C2"
- board text added: "I2C5"
- board text added: "Impedance Control:"
- board text added: "Min hole diameter:"
- board text added: "Min track/spacing:"
- board text added: "No"
- board text added: "None"
- board text added: "PWM"
- board text added: "Plated Board Edge:"
- board text added: "RST"
- board text added: "SPI1"
- board text added: "SPI2"
- board text added: "SWD"
- board text added: "Scott CJX"
- board text added: "UART10"
- board text added: "UART3"
- board text added: "USR1"
- board text added: "USR2"
- board text added: "V1"
- board text added: "V2"
- board text added: "VC G 5V G 3V3 06 07 08 09 10 11 12 12 14 15 16 17 18 19 20"
- board text added: "V_{1}"
- board text added: "V_{2}"
- board text added: "V_{BATT}"
