File: HDK/bigger-brain.kicad_pcb (KiCad board)
At the start: 4 copper layers, 100 x 100 mm, 109 parts, among them J301 TF-01A, J401 USB_C, J402 MicroFit_02x10V-H, J403 PH_01x05V-H, J404 PH_01x05V-H, J405 PH_01x05V-H, J406 PH_01x05V-H, J407 PH_01x05V-H, J408 PH_01x05V-H, J409 PH_01x05V-H, J410 PH_01x05V-H, J411 PH_01x05V-H, J412 PH_01x05V-H, J413 PHD_02x04V-H, J414 PHD_02x04V-H, J415 2.54mm2x20V-H, J416 PH_01x05V-H, J417 PHD_02x04V-H, SW401 SW_Push, SW402 SW_Push, SW403 SW_Push, SW404 SW_Push, U101 STM32H723ZGTx, U201 AMS1117-3.3, U203 AMS1117-5.0, U501 TJA1042T-3, U601 TJA1042T-3, U701 TJA1042T-3, X101 25MHz ±10ppm, Y101 32.768kHz 12.5pF ±20ppm

Commit message: freeze rev1.1
Parts:
- added R409: 10k, Resistor_SMD:R_0603_1608Metric, F.Cu at (93.2, 129.0)
Routing:
- net NRST: track 73.6 -> 76.4 mm
- net MCU-3.3V: track 147.8 -> 148.9 mm, vias 30 -> 31
Other:
- board text added: "Rev1.1"

Commit message: updated rev2
Parts:
- added D403: GREEN, LED_SMD:LED_0603_1608Metric, F.Cu at (116.4, 91.2)
- added D404: RED, LED_SMD:LED_0603_1608Metric, F.Cu at (116.4, 94.1)
- added D405: BLUE, LED_SMD:LED_0603_1608Metric, F.Cu at (116.4, 96.7)
- added D406: BLUE, LED_SMD:LED_0603_1608Metric, F.Cu at (50.2, 138.6)
- added J418: Generic Breakout, NVF-Kicad:PH_01x05V-H, F.Cu at (73.0, 76.2)
- added J419: Generic Breakout, NVF-Kicad:PH_01x05V-H, F.Cu at (78.5, 76.2)
- added J420: SPI Breakout, NVF-Kicad:PHD_02x04V-H, F.Cu at (85.0, 75.2)
- added J421: SPI Breakout, NVF-Kicad:PHD_02x04V-H, F.Cu at (62.5, 147.2)
- added J422: Generic Breakout, NVF-Kicad:PH_01x05V-H, F.Cu at (69.5, 148.2)
- added J423: UART Breakout, NVF-Kicad:PH_01x05V-H, F.Cu at (75.0, 148.2)
- added J424: UART Breakout, NVF-Kicad:PH_01x05V-H, F.Cu at (80.5, 148.2)
- added J425: Generic Breakout, NVF-Kicad:PH_01x05V-H, F.Cu at (86.0, 148.2)
- added J426: Generic Breakout, NVF-Kicad:PH_01x05V-H, F.Cu at (91.5, 148.2)
- added J427: SPI Breakout, NVF-Kicad:PHD_02x04V-H, F.Cu at (97.2, 147.2)
- added R410: 1k, Resistor_SMD:R_0603_1608Metric, F.Cu at (97.6, 66.1)
- added R411: 1k, Resistor_SMD:R_0603_1608Metric, F.Cu at (104.7, 66.1)
- added R412: 200, Resistor_SMD:R_0603_1608Metric, F.Cu at (113.0, 94.1)
- added R413: 200, Resistor_SMD:R_0603_1608Metric, F.Cu at (113.0, 96.7)
- added R414: 1k, Resistor_SMD:R_0603_1608Metric, F.Cu at (50.2, 140.5)
- F201, F202: footprint NVF-Kicad:FUSE-MCCQ-122 -> NVF-Kicad:FUSE-Littelfuse_Nano2_154x
- J403: value PH_01x05V-H -> 2.54mm2x20V-H; footprint NVF-Kicad:PH_01x05V-H -> NVF-Kicad:2.54mm2x20V-H
- J404, J405, J406, J410, J411, J412: value PH_01x05V-H -> Conn_01x02; footprint NVF-Kicad:PH_01x05V-H -> NVF-Kicad:PH_01x02V-H
- J407, J408, J409: value PH_01x05V-H -> I2C Breakout
- J413, J417: value PHD_02x04V-H -> Generic Breakout; footprint NVF-Kicad:PHD_02x04V-H -> NVF-Kicad:PH_01x05V-H
- J414: value PHD_02x04V-H -> UART Breakout; footprint NVF-Kicad:PHD_02x04V-H -> NVF-Kicad:PH_01x05V-H
- J415: value 2.54mm2x20V-H -> Generic Breakout; footprint NVF-Kicad:2.54mm2x20V-H -> NVF-Kicad:PH_01x05V-H
- J416: value PH_01x05V-H -> Generic Breakout
- R409: value 10k -> 200
- SWD401: footprint NVF-Kicad:2.54mm2x04V-H -> NVF-Kicad:PHD_02x04V-H
- moved J415 104.3 mm to (56.5, 76.2)
- moved J414 103.6 mm to (51.0, 76.2), turned to -90 degrees
- moved J408 99.6 mm to (73.0, 61.7), turned to -90 degrees
- moved J412 98.5 mm to (58.7, 65.2), turned to 0 degrees
- moved J407 93.6 mm to (67.5, 61.7), turned to -90 degrees
- moved J413 90.8 mm to (45.5, 76.2), turned to -90 degrees
- moved R102 79.6 mm to (63.9, 84.2), turned to 90 degrees
- moved R101 79.2 mm to (59.8, 84.2), turned to -90 degrees
- moved SWD401 78.7 mm to (85.0, 60.8), turned to 90 degrees
- moved J404 58.4 mm to (44.7, 58.2), turned to 0 degrees
- moved J403 52.7 mm to (84.7, 133.0), turned to -90 degrees
- moved SW402 51.1 mm to (55.0, 150.5), turned to 90 degrees
- moved J411 49.4 mm to (51.7, 65.2), turned to 0 degrees
- moved C401 49.2 mm to (55.0, 146.1)
- moved J410 47.5 mm to (44.7, 65.2), turned to 0 degrees
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Connections:
- J403 pad 1: PP-5.0V -> PG07
- J403 pad 2: MCU-3.3V -> PG08
- J403 pad 3: PE06 -> PG05
- J403 pad 4: PE05 -> PG06
- J403 pad 5: GND -> PG03
- J404 pad 1: PP-5.0V -> /CanTrx2/CAN_L
- J404 pad 2: MCU-3.3V -> /CanTrx2/CAN_H
- J405 pad 1: PP-5.0V -> /CanTrx1/CAN_L
- J405 pad 2: MCU-3.3V -> /CanTrx1/CAN_H
- J406 pad 1: PP-5.0V -> /CanTrx3/CAN_L
- J406 pad 2: MCU-3.3V -> /CanTrx3/CAN_H
- J407 pad 3: /UART2_TX -> /I2C5_SDA
- J407 pad 4: /UART2_RX -> /I2C5_SCL
- J408 pad 3: /UART3_TX -> /I2C5_SDA
- J408 pad 4: /UART3_RX -> /I2C5_SCL
- J409 pad 3: PE01 -> /I2C5_SDA
- J409 pad 4: PE00 -> /I2C5_SCL
- J410 pad 1: PP-5.0V -> /CanTrx2/CAN_L
- J410 pad 2: MCU-3.3V -> /CanTrx2/CAN_H
- J411 pad 1: PP-5.0V -> /CanTrx1/CAN_L
- J411 pad 2: MCU-3.3V -> /CanTrx1/CAN_H
- J412 pad 1: PP-5.0V -> /CanTrx3/CAN_L
- J412 pad 2: MCU-3.3V -> /CanTrx3/CAN_H
- J413 pad 2: PC04 -> MCU-3.3V
- J413 pad 3: MCU-3.3V -> PE06
- J413 pad 4: PA07 -> PE05
- J413 pad 5: PC05 -> GND
- J414 pad 2: /SPI2_SCLK -> MCU-3.3V
- J414 pad 3: MCU-3.3V -> /UART10_TX
- J414 pad 4: /SPI2_MOSI -> /UART10_RX
- J414 pad 5: /SPI2_IRQ -> GND
- J415 pad 1: PG07 -> PP-5.0V
- J415 pad 2: PG08 -> MCU-3.3V
- J415 pad 3: PG05 -> PF02
- J415 pad 4: PG06 -> PF03
- J415 pad 5: PG03 -> GND
- J416 pad 3: /UART10_TX -> PF02
- J416 pad 4: /UART10_RX -> PF03
- J417 pad 2: /SPI1_SCLK -> MCU-3.3V
- J417 pad 3: MCU-3.3V -> PB03
- J417 pad 4: /SPI1_MOSI -> PB04
- J417 pad 5: /SPI1_IRQ -> GND
- R101 pad 1: /I2C2_SCL -> /I2C5_SDA
- R102 pad 1: /I2C2_SDA -> /I2C5_SCL
- R409 pad 1: MCU-3.3V -> Net-(D403-K)
- R409 pad 2: NRST -> GND
- SW403 pad 1: USR_BTN1 -> Net-(R410-Pad2)
- SW404 pad 1: USR_BTN2 -> Net-(R411-Pad2)
- U101 pad 100: unconnected-(U101-PA8-Pad100) -> USR_LED
- U101 pad 127: unconnected-(U101-PG12-Pad127) -> PG12
- U101 pad 128: unconnected-(U101-PG13-Pad128) -> PG13
- U101 pad 133: unconnected-(U101-PB3(JTDO-Pad133) -> PB03
- U101 pad 134: unconnected-(U101-PB4(NJTRST)-Pad134) -> PB04
Routing:
- net VCC: track 130.3 -> 49.3 mm, vias 2 -> 3
- net /CanTrx3/CAN_H: track 17.3 -> 90.3 mm
- net /CanTrx3/CAN_L: track 15.0 -> 83.7 mm
- net /CanTrx1/CAN_H: track 17.4 -> 76.7 mm
- net PE09: track 35.5 -> 92.5 mm
- net /CanTrx1/CAN_L: track 15.0 -> 70.0 mm
- net /CanTrx2/CAN_H: track 17.2 -> 66.4 mm
- net /CanTrx2/CAN_L: track 15.0 -> 59.9 mm
- net /UART3_TX: track 46.4 -> 84.5 mm
- net /UART3_RX: track 48.9 -> 85.1 mm
- net /SWDIO: track 37.0 -> 69.6 mm, vias 1 -> 2
- net /SPI2_MISO: track 24.4 -> 56.9 mm, vias 0 -> 2
- net /SWCLK: track 47.6 -> 79.9 mm, vias 2 -> 3
- net /SPI2_MOSI: track 27.6 -> 59.5 mm, vias 0 -> 2
- net /SPI2_CS: track 20.1 -> 51.5 mm, vias 0 -> 1
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Other:
- board text added: "Rev2"
- board text added: "USR"
- board text added: "VCC"
- board text removed: "01 02 03 04 05 06 07 08 09 10 11 12 12 14 15 16 17 18 19 20"
- board text removed: "ANA"
- board text removed: "ANA/ SPI1"
- board text removed: "ANA/ UART2"
- board text removed: "G CLK DIO 3V3"
- board text removed: "G TX RX 3V3"
- board text removed: "I2C2"
- board text removed: "I2C5"
- board text removed: "PWM"
- board text removed: "Rev1.1"
- board text removed: "SPI1"
- board text removed: "SPI2"
- board text removed: "UART10"
- board text removed: "UART3"
- board text removed: "VC G 5V G 3V3 06 07 08 09 10 11 12 12 14 15 16 17 18 19 20"

Commit message: freeze rev2
Parts:
- J404, J405, J406, J410, J411, J412: footprint NVF-Kicad:PH_01x02V-H -> Connector_JST:JST_PH_B2B-PH-K_1x02_P2.00mm_Vertical
Connections:
- J420 pad 4: /SPI1_MOSI -> /SPI1_MISO
- J420 pad 6: /SPI1_MISO -> /SPI1_MOSI
- J427 pad 4: /SPI2_MOSI -> /SPI2_MISO
- J427 pad 6: /SPI2_MISO -> /SPI2_MOSI
Routing:
- net VCC: track 49.3 -> 122.8 mm
- net PE09: track 92.5 -> 20.0 mm
- net /SPI1_MOSI: track 20.1 -> 21.8 mm
- net /SPI1_MISO: track 21.3 -> 19.8 mm, vias 1 -> 0
- net /SPI2_MISO: track 56.9 -> 57.7 mm
Other:
- board text added: "Bigger-Brain Rev2"
- board text removed: "Bigger-Brain Rev1"
