File: HDK/bigger-brain.kicad_pcb (KiCad board)
At the start: 4 copper layers, 100 x 100 mm, 129 parts, among them J301 TF-01A, J401 USB_C, J402 MicroFit_02x10V-H, J403 2.54mm2x20V-H, J404 Conn_01x02, J405 Conn_01x02, J406 Conn_01x02, J407 I2C Breakout, J408 I2C Breakout, J409 I2C Breakout, J410 Conn_01x02, J411 Conn_01x02, J412 Conn_01x02, J413 Generic Breakout, J414 UART Breakout, J415 Generic Breakout, J416 Generic Breakout, J417 Generic Breakout, J418 Generic Breakout, J419 Generic Breakout, J420 SPI Breakout, J421 SPI Breakout, J422 Generic Breakout, J423 UART Breakout, J424 UART Breakout, J425 Generic Breakout, J426 Generic Breakout, J427 SPI Breakout, SW401 SW_Push, SW402 SW_Push, SW403 SW_Push, SW404 SW_Push, U101 STM32H723ZGTx, U201 AMS1117-3.3, U203 AMS1117-5.0, U501 TJA1042T-3, U601 TJA1042T-3, U701 TJA1042T-3, X101 25MHz ±10ppm, Y101 32.768kHz 12.5pF ±20ppm

Commit message: updated rev2.1
Parts:
- added JP401: Jumper_2_Open, Connector_PinHeader_2.54mm:PinHeader_1x02_P2.54mm_Vertical, F.Cu at (108.8, 94.2)
Routing:
- net VBUS: track 23.5 -> 35.2 mm
- net PB03: track 25.1 -> 26.4 mm
- net PA06: track 41.0 -> 40.2 mm
- net /CanTrx2/CAN_H: track 66.4 -> 67.1 mm
Other:
- board text added: "Bigger-Brain Rev2.1"
- board text added: "Rev2.1"
- board text added: "V_{USB} = V_{CC}"
- board text removed: "Bigger-Brain Rev2"
- board text removed: "Rev2"

Commit message: added fab and ibom
Parts:
- J402: value MicroFit_02x10V-H -> Molex_Micro-Fit_3.0_43045-2012_2x10_P3.00mm_Vertical
- J403: value 2.54mm2x20V-H -> 2x20V-H
- J404, J405, J406, J410, J411, J412: footprint Connector_JST:JST_PH_B2B-PH-K_1x02_P2.00mm_Vertical -> NVF-Kicad:PH_01x02V-H
- R409, R412, R413: value 200 -> 300
