File: HDK/CanTrx.kicad_sch (KiCad schematic)
At the start: 4 parts, among them U501 TJA1042T-3

Commit message: added rev1-final
Parts:
- removed R501: 10k, Resistor_SMD:R_0603_1608Metric, symbol Device:R
- C501, C502: LCSC C57112 -> C14663
Connections:
- net CAN_STB is gone; now on net GND: U501.8 (STB)
Other:
- company: (none) -> Scott CJX
- title: (none) -> Bigger Brain
Changed lines of the file:
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@@
 (kicad_sch (version 20230121) (generator eeschema)
   (paper "A4")
-  (junction (at 52.07 41.91) (diameter 0) (color 0 0 0 0)
+  (title_block
+    (title "Bigger Brain")
+    (date "2024-01-31")
+    (rev "1")
+    (company "Scott CJX")
   )
   (junction (at 29.21 39.37) (diameter 0) (color 0 0 0 0)
   )
+  (wire (pts (xy 63.5 49.53) (xy 63.5 41.91))
+    (stroke (width 0) (type default))
+  )
   (wire (pts (xy 78.74 49.53) (xy 78.74 46.99))
     (stroke (width 0) (type default))
@@
     (stroke (width 0) (type default))
   )
-  (wire (pts (xy 49.53 41.91) (xy 52.07 41.91))
-    (stroke (width 0) (type default))
-  )
   (wire (pts (xy 78.74 25.4) (xy 78.74 26.67))
     (stroke (width 0) (type default))
@@
     (stroke (width 0) (type default))
   )
-  (wire (pts (xy 52.07 35.56) (xy 52.07 41.91))
-    (stroke (width 0) (type default))
-  )
-  (wire (pts (xy 52.07 25.4) (xy 52.07 27.94))
-    (stroke (width 0) (type default))
-  )
-  (wire (pts (xy 52.07 41.91) (xy 66.04 41.91))
+  (wire (pts (xy 63.5 41.91) (xy 66.04 41.91))
     (stroke (width 0) (type default))
   )
@@
     (effects (font (size 1.27 1.27)) (justify left))
   )
-  (hierarchical_label "CAN_STB" (shape input) (at 49.53 41.91 180) (fields_autoplaced)
-    (effects (font (size 1.27 1.27)) (justify right))
-  )
   (symbol (lib_id "Device:C") (at 17.78 44.45 0) (unit 1)
     (in_bom yes) (on_board yes) (dnp no)
@@
       (effects (font (size 1.27 1.27)) hide)
     )
-    (property "LCSC" "C57112" (at 17.78 44.45 0)
+    (property "LCSC" "C14663" (at 17.78 44.45 0)
       (effects (font (size 1.27 1.27)) hide)
     )
@@
     )
   )
+  (symbol (lib_id "power:GND") (at 63.5 49.53 0) (unit 1)
+    (in_bom yes) (on_board yes) (dnp no) (fields_autoplaced)
+    (property "Reference" "#PWR0503" (at 63.5 55.88 0)
+      (effects (font (size 1.27 1.27)) hide)
+    )
+    (property "Value" "GND" (at 63.5 54.61 0)
+      (effects (font (size 1.27 1.27)) hide)
+    )
+    (property "Footprint" "" (at 63.5 49.53 0)
+      (effects (font (size 1.27 1.27)) hide)
+    )
+    (property "Datasheet" "" (at 63.5 49.53 0)
+      (effects (font (size 1.27 1.27)) hide)
+    )
+    (pin "1")
+    (instances
+      (project "bigger-brain"
+        (path "/4f585eb3-0717-4acd-9fc1-ccc573c80f45/9d2b90d0-8569-4b07-81d3-8efd9a28d2a6"
+          (reference "#PWR0503") (unit 1)
+        )
+        (path "/4f585eb3-0717-4acd-9fc1-ccc573c80f45/d0ce514a-b9ea-4179-9171-f24c19f45ab3"
+          (reference "#PWR0603") (unit 1)
+        )
+        (path "/4f585eb3-0717-4acd-9fc1-ccc573c80f45/c3ad5ae8-6df1-47a3-95c0-e59ed927cc6d"
+          (reference "#PWR0703") (unit 1)
+        )
+      )
+    )
+  )
   (symbol (lib_id "power:+5V") (at 17.78 25.4 0) (unit 1)
     (in_bom yes) (on_board yes) (dnp no)
@@
     )
   )
-  (symbol (lib_id "Device:R") (at 52.07 31.75 0) (mirror y) (unit 1)
-    (in_bom yes) (on_board yes) (dnp no)
-    (property "Reference" "R501" (at 50.8 30.48 0)
-      (effects (font (size 1.27 1.27)) (justify left))
-    )
-    (property "Value" "10k" (at 50.8 33.02 0)
-      (effects (font (size 1.27 1.27)) (justify left))
-    )
-    (property "Footprint" "Resistor_SMD:R_0603_1608Metric" (at 53.848 31.75 90)
-      (effects (font (size 1.27 1.27)) hide)
-    )
-    (property "Datasheet" "~" (at 52.07 31.75 0)
-      (effects (font (size 1.27 1.27)) hide)
-    )
-    (property "LCSC" "C25804" (at 52.07 31.75 0)
-      (effects (font (size 1.27 1.27)) hide)
-    )
+  (symbol (lib_id "power:GND") (at 17.78 49.53 0) (unit 1)
+    (in_bom yes) (on_board yes) (dnp no) (fields_autoplaced)
+    (property "Reference" "#PWR0505" (at 17.78 55.88 0)
+      (effects (font (size 1.27 1.27)) hide)
+    )
+    (property "Value" "GND" (at 17.78 54.61 0)
+      (effects (font (size 1.27 1.27)) hide)
+    )
+    (property "Footprint" "" (at 17.78 49.53 0)
+      (effects (font (size 1.27 1.27)) hide)
+    )
+    (property "Datasheet" "" (at 17.78 49.53 0)
+      (effects (font (size 1.27 1.27)) hide)
+    )
+    (pin "1")
+    (instances
+      (project "bigger-brain"
+        (path "/4f585eb3-0717-4acd-9fc1-ccc573c80f45/9d2b90d0-8569-4b07-81d3-8efd9a28d2a6"
+          (reference "#PWR0505") (unit 1)
+        )
+        (path "/4f585eb3-0717-4acd-9fc1-ccc573c80f45/d0ce514a-b9ea-4179-9171-f24c19f45ab3"
+          (reference "#PWR0605") (unit 1)
+        )
+        (path "/4f585eb3-0717-4acd-9fc1-ccc573c80f45/c3ad5ae8-6df1-47a3-95c0-e59ed927cc6d"
+          (reference "#PWR0705") (unit 1)
+        )
+      )
+    )
+  )
+  (symbol (lib_id "Device:C") (at 29.21 44.45 0) (unit 1)
+    (in_bom yes) (on_board yes) (dnp no)
+    (property "Reference" "C502" (at 31.75 43.18 0)
+      (effects (font (size 1.27 1.27)) (justify left))
+    )
+    (property "Value" "100n" (at 31.75 45.72 0)
+      (effects (font (size 1.27 1.27)) (justify left))
+    )
+    (property "Footprint" "Capacitor_SMD:C_0603_1608Metric" (at 30.1752 48.26 0)
+      (effects (font (size 1.27 1.27)) hide)
+    )
+    (property "Datasheet" "~" (at 29.21 44.45 0)
+      (effects (font (size 1.27 1.27)) hide)
+    )
+    (property "LCSC" "C14663" (at 29.21 44.45 0)
+      (effects (font (size 1.27 1.27)) hide)
+    )
+    (pin "1")
     (pin "2")
-    (pin "1")
-    (instances
-      (project "bigger-brain"
-        (path "/4f585eb3-0717-4acd-9fc1-ccc573c80f45/9d2b90d0-8569-4b07-81d3-8efd9a28d2a6"
-          (reference "R501") (unit 1)
-        )
-        (path "/4f585eb3-0717-4acd-9fc1-ccc573c80f45/d0ce514a-b9ea-4179-9171-f24c19f45ab3"
-          (reference "R601") (unit 1)
-        )
-        (path "/4f585eb3-0717-4acd-9fc1-ccc573c80f45/c3ad5ae8-6df1-47a3-95c0-e59ed927cc6d"
-          (reference "R701") (unit 1)
-        )
-      )
-    )
-  )
-  (symbol (lib_id "power:GND") (at 17.78 49.53 0) (unit 1)
-    (in_bom yes) (on_board yes) (dnp no) (fields_autoplaced)
-    (property "Reference" "#PWR0505" (at 17.78 55.88 0)
-      (effects (font (size 1.27 1.27)) hide)
-    )
-    (property "Value" "GND" (at 17.78 54.61 0)
-      (effects (font (size 1.27 1.27)) hide)
-    )
-    (property "Footprint" "" (at 17.78 49.53 0)
-      (effects (font (size 1.27 1.27)) hide)
-    )
-    (property "Datasheet" "" (at 17.78 49.53 0)
-      (effects (font (size 1.27 1.27)) hide)
-    )
-    (pin "1")
-    (instances
-      (project "bigger-brain"
-        (path "/4f585eb3-0717-4acd-9fc1-ccc573c80f45/9d2b90d0-8569-4b07-81d3-8efd9a28d2a6"
-          (reference "#PWR0505") (unit 1)
-        )
-        (path "/4f585eb3-0717-4acd-9fc1-ccc573c80f45/d0ce514a-b9ea-4179-9171-f24c19f45ab3"
-          (reference "#PWR0605") (unit 1)
-        )
-        (path "/4f585eb3-0717-4acd-9fc1-ccc573c80f45/c3ad5ae8-6df1-47a3-95c0-e59ed927cc6d"
-          (reference "#PWR0705") (unit 1)
-        )
-      )
-    )
-  )
-  (symbol (lib_id "Device:C") (at 29.21 44.45 0) (unit 1)
-    (in_bom yes) (on_board yes) (dnp no)
-    (property "Reference" "C502" (at 31.75 43.18 0)
-      (effects (font (size 1.27 1.27)) (justify left))
-    )
-    (property "Value" "100n" (at 31.75 45.72 0)
-      (effects (font (size 1.27 1.27)) (justify left))
-    )
-    (property "Footprint" "Capacitor_SMD:C_0603_1608Metric" (at 30.1752 48.26 0)
-      (effects (font (size 1.27 1.27)) hide)
-    )
-    (property "Datasheet" "~" (at 29.21 44.45 0)
-      (effects (font (size 1.27 1.27)) hide)
-    )
-    (property "LCSC" "C57112" (at 29.21 44.45 0)
-      (effects (font (size 1.27 1.27)) hide)
-    )
-    (pin "1")
-    (pin "2")
     (instances
       (project "bigger-brain"
@@
     )
   )
-  (symbol (lib_id "power:+3V3") (at 52.07 25.4 0) (unit 1)
-    (in_bom yes) (on_board yes) (dnp no)
-    (property "Reference" "#PWR0503" (at 52.07 29.21 0)
-      (effects (font (size 1.27 1.27)) hide)
-    )
-    (property "Value" "+3V3" (at 52.07 21.59 0)
-      (effects (font (size 1.27 1.27)))
-    )
-    (property "Footprint" "" (at 52.07 25.4 0)
-      (effects (font (size 1.27 1.27)) hide)
-    )
-    (property "Datasheet" "" (at 52.07 25.4 0)
-      (effects (font (size 1.27 1.27)) hide)
-    )
-    (pin "1")
-    (instances
-      (project "bigger-brain"
-        (path "/4f585eb3-0717-4acd-9fc1-ccc573c80f45/9d2b90d0-8569-4b07-81d3-8efd9a28d2a6"
-          (reference "#PWR0503") (unit 1)
-        )
-        (path "/4f585eb3-0717-4acd-9fc1-ccc573c80f45/d0ce514a-b9ea-4179-9171-f24c19f45ab3"
-          (reference "#PWR0603") (unit 1)
-        )
-        (path "/4f585eb3-0717-4acd-9fc1-ccc573c80f45/c3ad5ae8-6df1-47a3-95c0-e59ed927cc6d"
-          (reference "#PWR0703") (unit 1)
-        )
-      )
+  (symbol (lib_id "NVF-Kicad:NVF-Logo") (at 264.16 177.8 0) (unit 1)
+    (in_bom yes) (on_board yes) (dnp no) (fields_autoplaced)
+    (property "Reference" "#G401" (at 264.16 149.1047 0)
+      (effects (font (size 1.27 1.27)) hide)
+    )
+    (property "Value" "LOGO" (at 264.16 206.4953 0)
+      (effects (font (size 1.27 1.27)) hide)
+    )
+    (property "Footprint" "" (at 264.16 177.8 0)
+      (effects (font (size 1.27 1.27)) hide)
+    )
+    (property "Datasheet" "" (at 264.16 177.8 0)
+      (effects (font (size 1.27 1.27)) hide)
+    )
+    (instances
+      (project "bigger-brain"
+        (path "/4f585eb3-0717-4acd-9fc1-ccc573c80f45/a2e49620-6bcb-48ed-bf4e-cee4a2fe5c52"
+          (reference "#G401") (unit 1)
+        )
+        (path "/4f585eb3-0717-4acd-9fc1-ccc573c80f45"
+          (reference "#G101") (unit 1)
+        )
+        (path "/4f585eb3-0717-4acd-9fc1-ccc573c80f45/9d2b90d0-8569-4b07-81d3-8efd9a28d2a6"
+          (reference "#G501") (unit 1)
+        )
+        (path "/4f585eb3-0717-4acd-9fc1-ccc573c80f45/d0ce514a-b9ea-4179-9171-f24c19f45ab3"
+          (reference "#G601") (unit 1)
+        )
+        (path "/4f585eb3-0717-4acd-9fc1-ccc573c80f45/c3ad5ae8-6df1-47a3-95c0-e59ed927cc6d"
+          (reference "#G701") (unit 1)
+        )
+      )

Commit message: freeze rev2
Parts:
- C501, C502, U501: Element14 (none) -> -
Changed lines of the file:
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@@
 			)
 		)
-		(property "Element14" ""
+		(property "Element14" "-"
 			(at 17.78 44.45 0)
 			(effects
@@
 			)
 		)
-		(property "Element14" ""
+		(property "Element14" "-"
 			(at 78.74 36.83 0)
 			(effects
@@
 			)
 		)
-		(property "Element14" ""
+		(property "Element14" "-"
 			(at 29.21 44.45 0)
 			(effects

Commit message: updated rev2.1
Parts:
- C501, C502, U501: Assemble (none) -> 1
Changed lines of the file:
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@@
 	(title_block
 		(title "Bigger Brain")
-		(date "2024-03-05")
-		(rev "2")
+		(date "2024-04-08")
+		(rev "2.1")
 		(company "Scott CJX")
 	)
@@
 			)
 		)
+		(property "Assemble" "1"
+			(at 17.78 44.45 0)
+			(effects
+				(font
+					(size 1.27 1.27)
+				)
+				(hide yes)
+			)
+		)
 		(pin "1"
 		)
@@
 			)
 		)
+		(property "Assemble" "1"
+			(at 78.74 36.83 0)
+			(effects
+				(font
+					(size 1.27 1.27)
+				)
+				(hide yes)
+			)
+		)
 		(pin "1"
 		)
@@
 			(at 29.21 44.45 0)
 			(effects
+				(font
+					(size 1.27 1.27)
+				)
+				(hide yes)
+			)
+		)
+		(property "Assemble" "1"
+			(at 29.21 44.45 0)
+			(effects
