File: HDK/SDCard.kicad_sch (KiCad schematic)
At the start: 9 parts, among them J301 Micro_SD_Card_Det1

Commit message: added rev1-final
Parts:
- C301: LCSC C57112 -> C14663
- J301: value Micro_SD_Card_Det1 -> TF-01A; footprint NVF-Kicad:TF-01A -> NVF-Kicad:TFCard_TF-01A; LCSC (none) -> C91145
Other:
- company: (none) -> Scott CJX
- title: (none) -> Bigger Brain
Changed lines of the file:
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@@
 (kicad_sch (version 20230121) (generator eeschema)
   (paper "A4")
+  (title_block
+    (title "Bigger Brain")
+    (date "2024-01-31")
+    (rev "1")
+    (company "Scott CJX")
+  )
   (junction (at 54.61 36.83) (diameter 0) (color 0 0 0 0)
   )
@@
   )
   (label "_SD_DET" (at 91.44 54.61 180) (fields_autoplaced)
-    (effects (font (size 1.27 1.27) bold italic) (justify right bottom))
+    (effects (font (size 1.27 1.27)) (justify right bottom))
   )
   (hierarchical_label "SD_DAT2" (shape input) (at 92.71 31.75 180) (fields_autoplaced)
@@
   (hierarchical_label "SD_DAT0" (shape input) (at 92.71 46.99 180) (fields_autoplaced)
     (effects (font (size 1.27 1.27)) (justify right))
+  )
+  (symbol (lib_id "NVF-Kicad:NVF-Logo") (at 264.16 177.8 0) (unit 1)
+    (in_bom yes) (on_board yes) (dnp no) (fields_autoplaced)
+    (property "Reference" "#G401" (at 264.16 149.1047 0)
+      (effects (font (size 1.27 1.27)) hide)
+    )
+    (property "Value" "LOGO" (at 264.16 206.4953 0)
+      (effects (font (size 1.27 1.27)) hide)
+    )
+    (property "Footprint" "" (at 264.16 177.8 0)
+      (effects (font (size 1.27 1.27)) hide)
+    )
+    (property "Datasheet" "" (at 264.16 177.8 0)
+      (effects (font (size 1.27 1.27)) hide)
+    )
+    (instances
+      (project "bigger-brain"
+        (path "/4f585eb3-0717-4acd-9fc1-ccc573c80f45/a2e49620-6bcb-48ed-bf4e-cee4a2fe5c52"
+          (reference "#G401") (unit 1)
+        )
+        (path "/4f585eb3-0717-4acd-9fc1-ccc573c80f45"
+          (reference "#G101") (unit 1)
+        )
+        (path "/4f585eb3-0717-4acd-9fc1-ccc573c80f45/6e1dda42-c136-4dd9-b10b-de1fe2020430"
+          (reference "#G301") (unit 1)
+        )
+      )
+    )
   )
   (symbol (lib_id "Device:R") (at 36.83 39.37 90) (unit 1)
@@
       (effects (font (size 1.27 1.27)))
     )
-    (property "Value" "Micro_SD_Card_Det1" (at 116.205 22.86 0)
-      (effects (font (size 1.27 1.27)))
-    )
-    (property "Footprint" "NVF-Kicad:TF-01A" (at 167.64 24.13 0)
+    (property "Value" "TF-01A" (at 116.205 22.86 0)
+      (effects (font (size 1.27 1.27)))
+    )
+    (property "Footprint" "NVF-Kicad:TFCard_TF-01A" (at 167.64 24.13 0)
       (effects (font (size 1.27 1.27)) hide)
     )
@@
       (effects (font (size 1.27 1.27)) hide)
     )
-    (property "LCSC" "" (at 115.57 41.91 0)
+    (property "LCSC" "C91145" (at 115.57 41.91 0)
       (effects (font (size 1.27 1.27)) hide)
     )
@@
       (effects (font (size 1.27 1.27)) hide)
     )
-    (property "LCSC" "C57112" (at 54.61 41.91 0)
-      (effects (font (size 1.27 1.27)) hide)
-    )
+    (property "LCSC" "C14663" (at 54.61 41.91 0)
+      (effects (font (size 1.27 1.27)) hide)
+    )

Commit message: freeze rev2
Parts:
- C301, C302, J301, R301, R302, R303, R304, R305, R306: Element14 (none) -> -
Changed lines of the file:
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@@
 			)
 		)
-		(property "Element14" ""
+		(property "Element14" "-"
 			(at 36.83 39.37 0)
 			(effects
@@
 			)
 		)
-		(property "Element14" ""
+		(property "Element14" "-"
 			(at 64.77 41.91 0)
 			(effects
@@
 			)
 		)
-		(property "Element14" ""
+		(property "Element14" "-"
 			(at 77.47 54.61 0)
 			(effects
@@
 			)
 		)
-		(property "Element14" ""
+		(property "Element14" "-"
 			(at 36.83 44.45 0)
 			(effects
@@
 			)
 		)
-		(property "Element14" ""
+		(property "Element14" "-"
 			(at 36.83 41.91 0)
 			(effects
@@
 			)
 		)
-		(property "Element14" ""
+		(property "Element14" "-"
 			(at 36.83 36.83 0)
 			(effects
@@
 			)
 		)
-		(property "Element14" ""
+		(property "Element14" "-"
 			(at 36.83 46.99 0)
 			(effects
@@
 			)
 		)
-		(property "Element14" ""
+		(property "Element14" "-"
 			(at 115.57 41.91 0)
 			(effects
@@
 			)
 		)
-		(property "Element14" ""
+		(property "Element14" "-"
 			(at 54.61 41.91 0)
 			(effects

Commit message: updated rev2.1
Parts:
- C301, C302, J301, R301, R302, R303, R304, R305, R306: Assemble (none) -> 1
Changed lines of the file:
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@@
 	(title_block
 		(title "Bigger Brain")
-		(date "2024-03-05")
-		(rev "2")
+		(date "2024-04-08")
+		(rev "2.1")
 		(company "Scott CJX")
 	)
@@
 			)
 		)
+		(property "Assemble" "1"
+			(at 36.83 39.37 0)
+			(effects
+				(font
+					(size 1.27 1.27)
+				)
+				(hide yes)
+			)
+		)
 		(pin "1"
 		)
@@
 			)
 		)
+		(property "Assemble" "1"
+			(at 64.77 41.91 0)
+			(effects
+				(font
+					(size 1.27 1.27)
+				)
+				(hide yes)
+			)
+		)
 		(pin "1"
 		)
@@
 			)
 		)
+		(property "Assemble" "1"
+			(at 77.47 54.61 0)
+			(effects
+				(font
+					(size 1.27 1.27)
+				)
+				(hide yes)
+			)
+		)
 		(pin "1"
 		)
@@
 			)
 		)
+		(property "Assemble" "1"
+			(at 36.83 44.45 0)
+			(effects
+				(font
+					(size 1.27 1.27)
+				)
+				(hide yes)
+			)
+		)
 		(pin "1"
 		)
@@
 			)
 		)
+		(property "Assemble" "1"
+			(at 36.83 41.91 0)
+			(effects
+				(font
+					(size 1.27 1.27)
+				)
+				(hide yes)
+			)
+		)
 		(pin "1"
 		)
@@
 			)
 		)
+		(property "Assemble" "1"
+			(at 36.83 36.83 0)
+			(effects
+				(font
+					(size 1.27 1.27)
+				)
+				(hide yes)
+			)
+		)
 		(pin "1"
 		)
@@
 			)
 		)
+		(property "Assemble" "1"
+			(at 36.83 46.99 0)
+			(effects
+				(font
+					(size 1.27 1.27)
+				)
+				(hide yes)
+			)
+		)
 		(pin "1"
 		)
@@
 		)
 		(property "Element14" "-"
+			(at 115.57 41.91 0)
+			(effects
+				(font
+					(size 1.27 1.27)
+				)
+				(hide yes)
+			)
+		)
+		(property "Assemble" "1"
 			(at 115.57 41.91 0)
 			(effects
@@
 			(at 54.61 41.91 0)
 			(effects
+				(font
+					(size 1.27 1.27)
+				)
+				(hide yes)
+			)
+		)
+		(property "Assemble" "1"
+			(at 54.61 41.91 0)
+			(effects
