File: HDK/bigger-brain.kicad_sch (KiCad schematic)
At the start: 6 parts, among them U101 STM32H723ZGTx, X101 25MHz ±10ppm, Y101 32.768kHz 12.5pF ±20ppm

Commit message: added rev1-final
Parts:
- added R101, R102: 5k1, Resistor_SMD:R_0603_1608Metric, symbol Device:R
- C101: LCSC C57112 -> C14663
Connections:
- net +3V3: now also R101.2, R102.2
- net UART10_TX: now reaches U101.1 (PE2)
- net I2C5_SDA: now reaches U101.10 (PF0)
- net UART1_TX: now reaches U101.101 (PA9)
- net UART1_RX: now reaches U101.102 (PA10)
- net I2C5_SCL: now reaches U101.11 (PF1)
- net SD1_DET: now reaches U101.110 (PA15(JTDI))
- net USR_BTN2: now reaches U101.114 (PD0)
- net USR_BTN1: now reaches U101.115 (PD1)
- net PF02: now reaches U101.12 (PF2)
- net SPI1_IRQ: now reaches U101.122 (PD6)
- net SPI1_MOSI: now reaches U101.123 (PD7)
- net SPI1_MISO: now reaches U101.124 (PG9)
- net SPI1_CS: now reaches U101.125 (PG10)
- net SPI1_SCLK: now reaches U101.126 (PG11)
- net PF03: now reaches U101.13 (PF3)
- net PF04: now reaches U101.14 (PF4)
- net PE00: now reaches U101.141 (PE0)
- net PE01: now reaches U101.142 (PE1)
- net PF05: now reaches U101.15 (PF5)
- net UART10_RX: now reaches U101.2 (PE3)
- net PE04: now reaches U101.3 (PE4)
- net V2_SENSE: now reaches U101.34 (PA0)
- net V1_SENSE: now reaches U101.35 (PA1)
- net UART2_TX: now reaches U101.36 (PA2)
- net UART2_RX: now reaches U101.37 (PA3)
- net PE05: now reaches U101.4 (PE5)
- net PA05: now reaches U101.41 (PA5)
- net PA06: now reaches U101.42 (PA6)
- net PA07: now reaches U101.43 (PA7)
- net PC04: now reaches U101.44 (PC4)
- net PC05: now reaches U101.45 (PC5)
- net PB00: now reaches U101.46 (PB0)
- net PB01: now reaches U101.47 (PB1)
- net PB02: now reaches U101.48 (PB2)
- net PF11: now reaches U101.49 (PF11)
- net PE06: now reaches U101.5 (PE6)
- net PF13: now reaches U101.53 (PF13)
- net PF14: now reaches U101.54 (PF14)
- net PF15: now reaches U101.55 (PF15)
- net PG00: now reaches U101.56 (PG0)
- net PG01: now reaches U101.57 (PG1)
- net PE07: now reaches U101.58 (PE7)
- net PE08: now reaches U101.59 (PE8)
- net PE09: now reaches U101.60 (PE9)
- net PE10: now reaches U101.63 (PE10)
- net PE11: now reaches U101.64 (PE11)
- net PE12: now reaches U101.65 (PE12)
- net PE13: now reaches U101.66 (PE13)
- net PE14: now reaches U101.67 (PE14)
- net SPI2_IRQ: now reaches U101.68 (PE15)
- net I2C2_SCL: now reaches U101.69 (PB10)
- net I2C2_SCL: now also R101.1
- net I2C2_SDA: now reaches U101.70 (PB11)
- net I2C2_SDA: now also R102.1
- net SPI2_CS: now reaches U101.73 (PB12)
- net SPI2_SCLK: now reaches U101.74 (PB13)
- net SPI2_MISO: now reaches U101.75 (PB14)
- net SPI2_MOSI: now reaches U101.76 (PB15)
- net UART3_TX: now reaches U101.77 (PD8)
- net UART3_RX: now reaches U101.78 (PD9)
- net PD10: now reaches U101.79 (PD10)
- net PD11: now reaches U101.80 (PD11)
- net PD12: now reaches U101.81 (PD12)
- net PD13: now reaches U101.82 (PD13)
- net PD14: now reaches U101.85 (PD14)
- net PD15: now reaches U101.86 (PD15)
- net PG02: now reaches U101.87 (PG2)
- net PG03: now reaches U101.88 (PG3)
- net PG04: now reaches U101.89 (PG4)
- net PG05: now reaches U101.90 (PG5)
- net PG06: now reaches U101.91 (PG6)
- net PG07: now reaches U101.92 (PG7)
- net PG08: now reaches U101.93 (PG8)
- no-connect marks 3 -> 25
Other:
- sheet CanTrx1 ports: added none; removed CAN_STB
- sheet CanTrx2 ports: added none; removed CAN_STB
- sheet CanTrx3 ports: added none; removed CAN_STB
- sheet HMI ports: added A0, A1, A2, A3, D0, D1, D2, D3, D4, D5, DBG_UART_RX, DBG_UART_TX, I2C2_SCL, I2C2_SDA, I2C5_SCL, I2C5_SDA, PWM1, PWM2, PWM3, PWM4, SPI1_CS, SPI1_IRQ, SPI1_MISO, SPI1_MOSI, SPI1_SCLK, SPI2_CS, SPI2_IRQ, SPI2_MISO, SPI2_MOSI, SPI2_SCLK, SWCLK, SWDIO, UART10_RX, UART10_TX, UART2_RX, UART2_TX, UART3_RX, UART3_TX; removed DET1_A, DET1_B, DET2_A, DET2_B, DET3_A, DET3_B
- sheet Power ports: added V1_SENSE, V2_SENSE; removed none
- note added: "BLOCKED"
- note added: "UNUSED"
- company: (none) -> Scott CJX
- title: (none) -> Bigger Brain
Changed lines of the file:
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@@
   (paper "A3")
   (title_block
-    (date "2024-01-14")
+    (title "Bigger Brain")
+    (date "2024-01-31")
+    (rev "1")
+    (company "Scott CJX")
   )

Commit message: updated rev2
Connections:
- net I2C2_SCL: no longer R101.1
- net I2C2_SDA: no longer R102.1
- net I2C5_SCL: now also R102.1
- net I2C5_SDA: now also R101.1
- net USR_LED: now reaches U101.100 (PA8)
- net PG12: now reaches U101.127 (PG12)
- net PG13: now reaches U101.128 (PG13)
- net PB03: now reaches U101.133 (PB3(JTDO)
- net PB04: now reaches U101.134 (PB4(NJTRST))
- no-connect marks 25 -> 20
Other:
- sheet HMI ports: added none; removed A2, A3, D0, D1, D2, D3, D4, D5
Changed lines of the file:
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@@
 	(title_block
 		(title "Bigger Brain")
-		(date "2024-02-21")
-		(rev "1.1")
+		(date "2024-03-05")
+		(rev "2")
 		(company "Scott CJX")
 	)

Commit message: freeze rev2
Parts:
- C101, C103, C104, R101, R102, U101, X101, Y101: Element14 (none) -> -

Commit message: updated rev2.1
Parts:
- C101, C103, C104, R101, R102, U101, X101, Y101: Assemble (none) -> 1
Changed lines of the file:
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@@
 	(title_block
 		(title "Bigger Brain")
-		(date "2024-03-05")
-		(rev "2")
+		(date "2024-04-08")
+		(rev "2.1")
 		(company "Scott CJX")
 	)
